File: PwSup.kicad_sch (KiCad schematic)
At the start: 14 parts

Commit message: Schem & lib upd
added audiojack symbol & added PREAMP cascade
Parts:
- added CE5: 100u, Capacitor_THT:CP_Radial_D6.3mm_P2.50mm, symbol Device:C_Polarized
- added R5: 100, Resistor_THT:R_Axial_DIN0207_L6.3mm_D2.5mm_P7.62mm_Horizontal, symbol Device:R
Connections:
- net GND: now also CE5.2
- net VA: now also R5.2
- new net VMu: CE5.1, R5.1
Other:
- note added: "block Mu"
