File: Cp.kicad_sch (KiCad schematic)
At the start: 64 parts, among them Q10 J201, Q11 J201, Q3 2SC1815, Q4 2SC1815, Q5 2SC1815, Q6 2SC1815, Q7 2SC1815, Q8 2SC1815, Q9 2SC1815, SW1 SW_Push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

Commit message: Schem upd
Tone Stack addded
Connections:
- net PREAMP_OUT: no longer R11.1, RV1.3, U1.2 (-)
- new net PREAMP: R11.1, RV1.3, U1.2 (-)
Other:
- moved on the sheet: Q3, R15, R17
Changed lines of the file:
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@@
 	)
 	(rectangle
-		(start 90.17 16.51)
+		(start 99.06 50.8)
+		(end 104.14 60.96)
+		(radius 2.54)
+		(stroke
+			(width 0.3048)
+			(type solid)
+			(color 255 153 0 1)
+		)
+		(fill
+			(type none)
+		)
+	)
+	(rectangle
+		(start 88.9 16.51)
 		(end 165.1 67.31)
 		(radius 4.064)
@@
 	)
 	(junction
-		(at 82.55 38.1)
-		(diameter 0)
-		(color 0 0 0 0)
-	)
-	(junction
 		(at 113.03 30.48)
 		(diameter 0)
@@
 	)
 	(junction
-		(at 71.12 38.1)
+		(at 102.87 45.72)
 		(diameter 0)
 		(color 0 0 0 0)
 	)
 	(junction
-		(at 97.79 30.48)
+		(at 71.12 38.1)
 		(diameter 0)
 		(color 0 0 0 0)
@@
 	)
 	(junction
-		(at 76.2 48.26)
+		(at 96.52 30.48)
 		(diameter 0)
 		(color 0 0 0 0)
 	)
 	(junction
-		(at 72.39 97.79)
+		(at 96.52 45.72)
 		(diameter 0)
 		(color 0 0 0 0)
 	)
 	(junction
-		(at 135.89 101.6)
+		(at 76.2 48.26)
 		(diameter 0)
 		(color 0 0 0 0)
 	)
 	(junction
-		(at 88.9 88.9)
+		(at 72.39 97.79)
 		(diameter 0)
 		(color 0 0 0 0)
 	)
 	(junction
-		(at 102.87 45.72)
+		(at 135.89 101.6)
+		(diameter 0)
+		(color 0 0 0 0)
+	)
+	(junction
+		(at 88.9 88.9)
 		(diameter 0)
 		(color 0 0 0 0)
@@
 	)
 	(junction
+		(at 82.55 38.1)
+		(diameter 0)
+		(color 0 0 0 0)
+	)
+	(junction
 		(at 81.28 97.79)
 		(diameter 0)
@@
 	)
 	(junction
-		(at 97.79 45.72)
-		(diameter 0)
-		(color 0 0 0 0)
-	)
-	(junction
 		(at 52.07 55.88)
 		(diameter 0)
@@
 	(wire
 		(pts
-			(xy 82.55 38.1) (xy 90.17 38.1)
-		)
-		(stroke
-			(width 0)
-			(type default)
-		)
-	)
-	(wire
-		(pts
 			(xy 76.2 38.1) (xy 82.55 38.1)
 		)
@@
 	(wire
 		(pts
+			(xy 82.55 38.1) (xy 88.9 38.1)
+		)
+		(stroke
+			(width 0)
+			(type default)
+		)
+	)
+	(wire
+		(pts
 			(xy 121.92 30.48) (xy 124.46 30.48)
 		)
@@
 	(wire
 		(pts
-			(xy 97.79 17.78) (xy 97.79 21.59)
+			(xy 96.52 17.78) (xy 96.52 21.59)
 		)
 		(stroke
@@
 	(wire
 		(pts
-			(xy 97.79 43.18) (xy 97.79 45.72)
+			(xy 96.52 43.18) (xy 96.52 45.72)
 		)
 		(stroke
@@
 	(wire
 		(pts
-			(xy 97.79 45.72) (xy 97.79 46.99)
+			(xy 96.52 45.72) (xy 96.52 46.99)
 		)
 		(stroke
@@
 	(wire
 		(pts
-			(xy 97.79 29.21) (xy 97.79 30.48)
+			(xy 96.52 29.21) (xy 96.52 30.48)
 		)
 		(stroke
@@
 	(wire
 		(pts
-			(xy 102.87 45.72) (xy 102.87 57.15)
+			(xy 102.87 45.72) (xy 102.87 59.69)
 		)
 		(stroke
@@
 	(wire
 		(pts
+			(xy 96.52 30.48) (xy 102.87 30.48)
+		)
+		(stroke
+			(width 0)
+			(type default)
+		)
+	)
+	(wire
+		(pts
 			(xy 132.08 38.1) (xy 132.08 40.64)
 		)
@@
 	(wire
 		(pts
-			(xy 97.79 30.48) (xy 97.79 33.02)
+			(xy 96.52 30.48) (xy 96.52 33.02)
 		)
 		(stroke
@@
 	(wire
 		(pts
-			(xy 102.87 45.72) (xy 97.79 45.72)
-		)
-		(stroke
-			(width 0)
-			(type default)
-		)
-	)
-	(wire
-		(pts
 			(xy 156.21 88.9) (xy 158.75 88.9)
 		)
@@
 	(wire
 		(pts
-			(xy 102.87 30.48) (xy 97.79 30.48)
+			(xy 81.28 102.87) (xy 81.28 106.68)
 		)
 		(stroke
@@
 	(wire
 		(pts
-			(xy 81.28 102.87) (xy 81.28 106.68)
+			(xy 121.92 29.21) (xy 121.92 30.48)
 		)
 		(stroke
@@
 	(wire
 		(pts
-			(xy 121.92 29.21) (xy 121.92 30.48)
+			(xy 59.69 25.4) (xy 59.69 30.48)
 		)
 		(stroke
@@
 	(wire
 		(pts
-			(xy 59.69 25.4) (xy 59.69 30.48)
+			(xy 29.21 40.64) (xy 29.21 35.56)
 		)
 		(stroke
@@
 	(wire
 		(pts
-			(xy 29.21 40.64) (xy 29.21 35.56)
+			(xy 96.52 45.72) (xy 102.87 45.72)
 		)
 		(stroke
@@
 	)
 	(label "VC"
-		(at 97.79 17.78 270)
+		(at 96.52 17.78 270)
 		(effects
 			(font
@@
 		)
 	)
-	(label "PREAMP_OUT"
+	(label "PREAMP"
 		(at 21.59 35.56 0)
 		(effects
@@
 	)
 	(label "CP_OUT"
-		(at 102.87 57.15 90)
+		(at 102.87 59.69 90)
 		(effects
 			(font
@@
 	(symbol
 		(lib_id "Transistor_BJT:2SC1815")
-		(at 95.25 38.1 0)
+		(at 93.98 38.1 0)
 		(unit 1)
 		(body_style 1)
@@
 		(dnp no)
 		(property "Reference" "Q3"
-			(at 99.568 36.83 0)
+			(at 98.298 36.83 0)
 			(show_name no)
 			(do_not_autoplace no)
@@
 		)
 		(property "Value" "2SC1815"
-			(at 99.568 39.37 0)
+			(at 98.298 39.37 0)
 			(show_name no)
 			(do_not_autoplace no)
@@
 		)
 		(property "Footprint" "Package_TO_SOT_THT:TO-92_Inline"
-			(at 100.33 40.005 0)
+			(at 99.06 40.005 0)
 			(hide yes)
 			(show_name no)
@@
 		)
 		(property "Datasheet" "https://media.digikey.com/pdf/Data%20Sheets/Toshiba%20PDFs/2SC1815.pdf"
-			(at 95.25 38.1 0)
+			(at 93.98 38.1 0)
 			(hide yes)
 			(show_name no)
@@
 		)
 		(property "Description" "0.15A Ic, 50V Vce, Low Noise Audio NPN Transistor, TO-92"
-			(at 95.25 38.1 0)
+			(at 93.98 38.1 0)
 			(hide yes)
 			(show_name no)
@@
 		)
 		(property "Sim.Device" "NPN"
-			(at 95.25 38.1 0)
+			(at 93.98 38.1 0)
 			(hide yes)
 			(show_name no)
@@
 		)
 		(property "Sim.Pins" "1=E 2=C 3=B"
-			(at 95.25 38.1 0)
+			(at 93.98 38.1 0)
 			(hide yes)
 			(show_name no)
@@
 	(symbol
 		(lib_id "Device:R")
-		(at 97.79 25.4 0)
+		(at 96.52 25.4 0)
 		(unit 1)
 		(body_style 1)
@@
 		(dnp no)
 		(property "Reference" "R17"
-			(at 99.06 24.13 0)
+			(at 97.79 24.13 0)
 			(show_name no)
 			(do_not_autoplace no)
@@
 		)
 		(property "Value" "10K"
-			(at 99.06 26.416 0)
+			(at 97.79 26.416 0)
 			(show_name no)
 			(do_not_autoplace no)
@@
 		)
 		(property "Footprint" ""
-			(at 96.012 25.4 90)
+			(at 94.742 25.4 90)
 			(hide yes)
 			(show_name no)
@@
 		)
 		(property "Datasheet" ""
-			(at 97.79 25.4 0)
+			(at 96.52 25.4 0)
 			(hide yes)
 			(show_name no)
@@
 		)
 		(property "Description" "Resistor"
-			(at 97.79 25.4 0)
+			(at 96.52 25.4 0)
 			(hide yes)
 			(show_name no)
@@
 	(symbol
 		(lib_id "power:GND")
-		(at 97.79 54.61 0)
+		(at 96.52 54.61 0)
 		(unit 1)
 		(body_style 1)
@@
 		(fields_autoplaced yes)
 		(property "Reference" "#PWR017"
-			(at 97.79 60.96 0)
+			(at 96.52 60.96 0)
 			(hide yes)
 			(show_name no)
@@
 		)
 		(property "Value" "GND"
-			(at 97.79 59.69 0)
+			(at 96.52 59.69 0)
 			(hide yes)
 			(show_name no)
@@
 		)
 		(property "Footprint" ""
-			(at 97.79 54.61 0)
+			(at 96.52 54.61 0)
 			(hide yes)
 			(show_name no)
@@
 		)
 		(property "Datasheet" ""
-			(at 97.79 54.61 0)
+			(at 96.52 54.61 0)
 			(hide yes)
 			(show_name no)
@@
 		)
 		(property "Description" "Power symbol creates a global label with name \"GND\" , ground"
-			(at 97.79 54.61 0)
+			(at 96.52 54.61 0)
 			(hide yes)
 			(show_name no)
@@
 	(symbol
 		(lib_id "Device:R")
-		(at 97.79 50.8 0)
+		(at 96.52 50.8 0)
 		(mirror y)
 		(unit 1)
@@
 		(dnp no)
 		(property "Reference" "R15"
-			(at 96.52 49.53 0)
+			(at 95.25 49.53 0)
 			(show_name no)
 			(do_not_autoplace no)
@@
 		)
 		(property "Value" "10K"
-			(at 96.52 51.816 0)
+			(at 95.25 51.816 0)
 			(show_name no)
 			(do_not_autoplace no)
@@
 		)
 		(property "Footprint" ""
-			(at 99.568 50.8 90)
+			(at 98.298 50.8 90)
 			(hide yes)
 			(show_name no)
@@
 		)
 		(property "Datasheet" ""
-			(at 97.79 50.8 0)
+			(at 96.52 50.8 0)
 			(hide yes)
 			(show_name no)
@@
 		)
 		(property "Description" "Resistor"
-			(at 97.79 50.8 0)
+			(at 96.52 50.8 0)
 			(hide yes)
 			(show_name no)
