File: AMP-MA.kicad_sch (KiCad schematic)
At the start: 54 parts, among them J8 Conn_01x05_Socket, Q1 2N5484, Q12 2N5484, Q13 2N5484, Q2 2N5484, U2 LM1875, U3 TL072

Commit message: smal schem upd
Parts:
- R39, R46: value 5K -> 4K7
- R54: value 10K -> 4K7
Other:
- moved on the sheet: C34, C6, CE6, CE7, R50, U2
