File: AMP-MA.kicad_sch (KiCad schematic)
At the start: 54 parts, among them J8 Conn_01x05_Socket, Q1 2N5484, Q12 2N5484, Q13 2N5484, Q2 2N5484, U2 LM1875, U3 TL072

Commit message: PCB and Schem upd
Parts:
- added unit 2 of U3
Connections:
- no-connect marks 0 -> 3
Changed lines of the file:
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@@
 	)
 	(junction
+		(at 44.45 16.51)
+		(diameter 0)
+		(color 0 0 0 0)
+	)
+	(junction
 		(at 59.69 29.21)
 		(diameter 0)
@@
 		(color 0 0 0 0)
 	)
+	(no_connect
+		(at 148.59 118.11)
+	)
+	(no_connect
+		(at 163.83 120.65)
+	)
+	(no_connect
+		(at 148.59 123.19)
+	)
 	(wire
 		(pts
@@
 	(wire
 		(pts
-			(xy 68.58 114.3) (xy 78.74 114.3)
+			(xy 68.58 114.3) (xy 73.66 114.3)
 		)
 		(stroke
@@
 	(wire
 		(pts
-			(xy 44.45 16.51) (xy 59.69 16.51)
+			(xy 39.37 16.51) (xy 44.45 16.51)
 		)
 		(stroke
@@
 	(wire
 		(pts
+			(xy 44.45 16.51) (xy 59.69 16.51)
+		)
+		(stroke
+			(width 0)
+			(type default)
+		)
+	)
+	(wire
+		(pts
 			(xy 78.74 30.48) (xy 78.74 29.21)
 		)
@@
 	(wire
 		(pts
-			(xy 101.6 19.05) (xy 115.57 19.05)
+			(xy 109.22 19.05) (xy 115.57 19.05)
 		)
 		(stroke
@@
 		)
 	)
-	(label "PREAMP1"
-		(at 92.71 34.29 180)
+	(label "VCC"
+		(at 204.47 49.53 0)
 		(effects
 			(font
 				(size 1.27 1.27)
 			)
-			(justify right bottom)
+			(justify left bottom)
 		)
 	)
-	(label "VCC"
-		(at 133.35 59.69 270)
+	(label "PREAMP1"
+		(at 92.71 34.29 180)
 		(effects
 			(font
@@
 		)
 	)
-	(label "PREAMP"
-		(at 78.74 114.3 180)
+	(label "VCC"
+		(at 133.35 59.69 270)
 		(effects
 			(font
@@
 	)
 	(label "VEE"
-		(at 120.65 128.27 90)
+		(at 215.9 49.53 0)
 		(effects
 			(font
@@
 		)
 	)
-	(label "ToneSt"
-		(at 100.33 71.12 0)
+	(label "VEE"
+		(at 120.65 128.27 90)
 		(effects
 			(font
@@
 		)
 	)
-	(label "LM_OUT"
-		(at 144.78 73.66 0)
+	(label "ToneSt"
+		(at 100.33 71.12 0)
 		(effects
 			(font
@@
 		)
 	)
-	(label "CP_OUT"
-		(at 101.6 19.05 0)
+	(label "LM_OUT"
+		(at 144.78 73.66 0)
 		(effects
 			(font
@@
 		)
 	)
+	(global_label "CP_OUT"
+		(shape input)
+		(at 109.22 19.05 180)
+		(fields_autoplaced yes)
+		(effects
+			(font
+				(size 1.27 1.27)
+			)
+			(justify right)
+		)
+		(property "Intersheetrefs" "${INTERSHEET_REFS}"
+			(at 99.0986 19.05 0)
+			(hide yes)
+			(show_name no)
+			(do_not_autoplace no)
+			(effects
+				(font
+					(size 1.27 1.27)
+				)
+				(justify right)
+			)
+		)
+	)
+	(global_label "VMu"
+		(shape input)
+		(at 39.37 16.51 180)
+		(fields_autoplaced yes)
+		(effects
+			(font
+				(size 1.27 1.27)
+			)
+			(justify right)
+		)
+		(property "Intersheetrefs" "${INTERSHEET_REFS}"
+			(at 32.6958 16.51 0)
+			(hide yes)
+			(show_name no)
+			(do_not_autoplace no)
+			(effects
+				(font
+					(size 1.27 1.27)
+				)
+				(justify right)
+			)
+		)
+	)
+	(global_label "PREAMP"
+		(shape input)
+		(at 73.66 114.3 0)
+		(fields_autoplaced yes)
+		(effects
+			(font
+				(size 1.27 1.27)
+			)
+			(justify left)
+		)
+		(property "Intersheetrefs" "${INTERSHEET_REFS}"
+			(at 84.1442 114.3 0)
+			(hide yes)
+			(show_name no)
+			(do_not_autoplace no)
+			(effects
+				(font
+					(size 1.27 1.27)
+				)
+				(justify left)
+			)
+		)
+	)
+	(global_label "VEE"
+		(shape input)
+		(at 215.9 49.53 180)
+		(fields_autoplaced yes)
+		(effects
+			(font
+				(size 1.27 1.27)
+			)
+			(justify right)
+		)
+		(property "Intersheetrefs" "${INTERSHEET_REFS}"
+			(at 209.5282 49.53 0)
+			(hide yes)
+			(show_name no)
+			(do_not_autoplace no)
+			(effects
+				(font
+					(size 1.27 1.27)
+				)
+				(justify right)
+			)
+		)
+	)
+	(global_label "VCC"
+		(shape input)
+		(at 204.47 49.53 180)
+		(fields_autoplaced yes)
+		(effects
+			(font
+				(size 1.27 1.27)
+			)
+			(justify right)
+		)
+		(property "Intersheetrefs" "${INTERSHEET_REFS}"
+			(at 197.8562 49.53 0)
+			(hide yes)
+			(show_name no)
+			(do_not_autoplace no)
+			(effects
+				(font
+					(size 1.27 1.27)
+				)
+				(justify right)
+			)
+		)
+	)
 	(symbol
 		(lib_id "Device:R_Potentiometer")
@@
 				)
 			)
+		)
+	)
+	(symbol
+		(lib_id "Amplifier_Operational:TL072")
+		(at 156.21 120.65 0)
+		(unit 2)
+		(body_style 1)
+		(exclude_from_sim no)
+		(in_bom yes)
+		(on_board yes)
+		(in_pos_files yes)
+		(dnp no)
+		(property "Reference" "U3"
+			(at 156.21 110.49 0)
+			(show_name no)
+			(do_not_autoplace no)
+			(effects
+				(font
+					(size 1.27 1.27)
+				)
+			)
+		)
+		(property "Value" "TL072"
+			(at 156.21 113.03 0)
+			(show_name no)
+			(do_not_autoplace no)
+			(effects
+				(font
+					(size 1.27 1.27)
+				)
+			)
+		)
+		(property "Footprint" ""
+			(at 156.21 120.65 0)
+			(hide yes)
+			(show_name no)
+			(do_not_autoplace no)
+			(effects
+				(font
+					(size 1.27 1.27)
+				)
+			)
+		)
+		(property "Datasheet" "http://www.ti.com/lit/ds/symlink/tl071.pdf"
+			(at 156.21 120.65 0)
+			(hide yes)
+			(show_name no)
+			(do_not_autoplace no)
+			(effects
+				(font
+					(size 1.27 1.27)
+				)
+			)
+		)
+		(property "Description" "Dual Low-Noise JFET-Input Operational Amplifiers, DIP-8/SOIC-8"
+			(at 156.21 120.65 0)
+			(hide yes)
+			(show_name no)
+			(do_not_autoplace no)
+			(effects
+				(font
+					(size 1.27 1.27)
+				)
+			)
+		)
+		(pin "6"
+		)
+		(pin "5"
+		)
+		(pin "1"
+		)
+		(pin "2"
+		)
+		(pin "3"
+		)
+		(pin "7"
+		)
+		(pin "4"
+		)
+		(pin "8"
+		)
+		(instances
+			(project "AMP-MA"
+				(path "/4094031b-a9da-4ac5-aaa1-42b342c92a3e"
+					(reference "U3")
+					(unit 2)
+				)
+			)

Commit message: Big upd
fully routed pcb. Some small updates for Schematic
Parts:
- added J9: Socket_01x03, Connector_JST:JST_XH_B3B-XH-A_1x03_P2.50mm_Vertical, symbol Connector:Conn_01x03_Socket
- C2, C24, C25, C26, C27, C28, C29, C3, C30, C31, C32, C33, C34, C35, C4, C5, C6: footprint Capacitor_THT:C_Disc_D7.0mm_W2.5mm_P5.00mm -> PrLib:C_disc_D7_W2.5_P5
- J8: value Conn_01x05_Socket -> Socket_01x05; footprint Connector_JST:JST_PH_B5B-PH-K_1x05_P2.00mm_Vertical -> Connector_JST:JST_XH_B5B-XH-A_1x05_P2.50mm_Vertical
- R62: renamed from R50; value 20K -> 22K
- RBass1, RMiddle1, RTreble1, VOL1, VOL2: footprint Potentiometer_THT:Potentiometer_Alps_RK09Y11_Single_Horizontal -> PrLib:potentiometer
- U3: footprint (none) -> Package_DIP:DIP-8_W7.62mm
- renumbered R6 to R10, R7 to R11, R38 to R12, R8 to R13, R9 to R14, R40 to R15, R44 to R16, R45 to R17, R42 to R18, R41 to R19, R54 to R20, R46 to R21, R39 to R22, R48 to R55, R52 to R60, R51 to R61, R47 to R63, R49 to R64
Connections:
- net GND: now also J9.2 (Pin_2); no longer LS1.1
- net LM_OUT: now also J9.1 (Pin_1)
- new net: J9.3 (Pin_3), LS1.1
Other:
- moved on the sheet: LS1

Commit message: small upd
changed & added capacitor footprint. replaced potentimeters
Parts:
- renumbered RBass1 to Bass1, RMiddle1 to Middle1, RTreble1 to Treble1
Changed lines of the file:
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@@
 		(in_pos_files yes)
 		(dnp no)
-		(property "Reference" "RBass1"
+		(property "Reference" "Bass1"
 			(at 132.08 35.56 0)
 			(show_name no)
@@
 			(project "AMP-MA"
 				(path "/4094031b-a9da-4ac5-aaa1-42b342c92a3e"
-					(reference "RBass1")
+					(reference "Bass1")
 					(unit 1)
 				)
@@
 		(in_pos_files yes)
 		(dnp no)
-		(property "Reference" "RTreble1"
+		(property "Reference" "Treble1"
 			(at 132.08 24.13 0)
 			(show_name no)
@@
 			(project "AMP-MA"
 				(path "/4094031b-a9da-4ac5-aaa1-42b342c92a3e"
-					(reference "RTreble1")
+					(reference "Treble1")
 					(unit 1)
 				)
@@
 		(in_pos_files yes)
 		(dnp no)
-		(property "Reference" "RMiddle1"
+		(property "Reference" "Middle1"
 			(at 134.62 43.18 0)
 			(show_name no)
@@
 			(project "AMP-MA"
 				(path "/4094031b-a9da-4ac5-aaa1-42b342c92a3e"
-					(reference "RMiddle1")
-					(unit 1)
-				)
+					(reference "Middle1")
+					(unit 1)
+				)

Commit message: First Beta
Parts:
- added GND1: MountingHole_Pad, MountingHole:MountingHole_2.2mm_M2_DIN965_Pad, symbol Mechanical:MountingHole_Pad
- added H1, H2: MountingHole, MountingHole:MountingHole_2.2mm_M2, symbol Mechanical:MountingHole
Connections:
- net GND: now also GND1.1

Commit message: Dev(#4)
* Patch 0

PCB updates

* Patch 1

Major PCB update

* Delete AMP-MA-backups directory

* Patch 2 gitignore update

PCB update

* Repository cleaned up

* PCB upd

Traces upd, created net classes

* Beta Version 0.0.1

Traces upd, Readme Upd
Parts:
- renumbered Q13 to Q3, Q12 to Q4
Connections:
- net U3_3: now reaches R21.2, R22.2, U3.3 (+)
Other:
- moved on the sheet: C25, C30, R15
Changed lines of the file:
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@@
 	)
 	(junction
-		(at 45.72 36.83)
+		(at 46.99 36.83)
 		(diameter 0)
 		(color 0 0 0 0)
@@
 	)
 	(junction
-		(at 45.72 78.74)
+		(at 46.99 78.74)
 		(diameter 0)
 		(color 0 0 0 0)
@@
 	)
 	(junction
-		(at 45.72 50.8)
+		(at 46.99 50.8)
 		(diameter 0)
 		(color 0 0 0 0)
@@
 	)
 	(junction
-		(at 45.72 92.71)
+		(at 46.99 92.71)
 		(diameter 0)
 		(color 0 0 0 0)
@@
 	(wire
 		(pts
-			(xy 45.72 78.74) (xy 53.34 78.74)
-		)
-		(stroke
-			(width 0)
-			(type default)
-		)
-	)
-	(wire
-		(pts
 			(xy 158.75 67.31) (xy 158.75 73.66)
 		)
@@
 	(wire
 		(pts
-			(xy 54.61 50.8) (xy 45.72 50.8)
-		)
-		(stroke
-			(width 0)
-			(type default)
-		)
-	)
-	(wire
-		(pts
 			(xy 59.69 16.51) (xy 59.69 17.78)
 		)
@@
 	(wire
 		(pts
-			(xy 45.72 36.83) (xy 52.07 36.83)
-		)
-		(stroke
-			(width 0)
-			(type default)
-		)
-	)
-	(wire
-		(pts
 			(xy 29.21 71.12) (xy 29.21 73.66)
 		)
@@
 	(wire
 		(pts
-			(xy 40.64 87.63) (xy 40.64 92.71)
+			(xy 40.64 88.9) (xy 40.64 92.71)
 		)
 		(stroke
@@
 	(wire
 		(pts
-			(xy 45.72 38.1) (xy 45.72 36.83)
+			(xy 46.99 38.1) (xy 46.99 36.83)
 		)
 		(stroke
@@
 	(wire
 		(pts
-			(xy 45.72 92.71) (xy 55.88 92.71)
-		)
-		(stroke
-			(width 0)
-			(type default)
-		)
-	)
-	(wire
-		(pts
 			(xy 118.11 95.25) (xy 120.65 95.25)
 		)
@@
 	(wire
 		(pts
-			(xy 40.64 92.71) (xy 45.72 92.71)
+			(xy 40.64 92.71) (xy 55.88 92.71)
 		)
 		(stroke
@@
 	(wire
 		(pts
-			(xy 45.72 80.01) (xy 45.72 78.74)
+			(xy 46.99 81.28) (xy 46.99 78.74)
 		)
 		(stroke
@@
 	(wire
 		(pts
-			(xy 40.64 78.74) (xy 40.64 80.01)
+			(xy 40.64 78.74) (xy 40.64 81.28)
 		)
 		(stroke
@@
 	(wire
 		(pts
-			(xy 45.72 87.63) (xy 45.72 92.71)
+			(xy 46.99 88.9) (xy 46.99 92.71)
 		)
 		(stroke
@@
 	(wire
 		(pts
-			(xy 45.72 45.72) (xy 45.72 50.8)
+			(xy 46.99 45.72) (xy 46.99 50.8)
 		)
 		(stroke
@@
 	(wire
 		(pts
-			(xy 40.64 78.74) (xy 45.72 78.74)
+			(xy 40.64 78.74) (xy 53.34 78.74)
 		)
 		(stroke
@@
 	(wire
 		(pts
-			(xy 40.64 50.8) (xy 45.72 50.8)
+			(xy 40.64 50.8) (xy 54.61 50.8)
 		)
 		(stroke
@@
 	(wire
 		(pts
-			(xy 40.64 36.83) (xy 45.72 36.83)
+			(xy 40.64 36.83) (xy 52.07 36.83)
 		)
 		(stroke
@@
 		)
 	)
+	(label "U3_3"
+		(at 45.72 111.76 0)
+		(effects
+			(font
+				(size 1.27 1.27)
+			)
+			(justify left bottom)
+		)
+	)
 	(label "LM_IN+"
 		(at 121.92 71.12 0)
@@
 	(symbol
 		(lib_id "Device:C")
-		(at 45.72 83.82 180)
+		(at 46.99 85.09 0)
+		(mirror x)
 		(unit 1)
 		(body_style 1)
@@
 		(dnp no)
 		(property "Reference" "C30"
-			(at 45.974 81.788 0)
+			(at 46.736 83.058 0)
 			(show_name no)
 			(do_not_autoplace no)
@@
 		)
 		(property "Value" "10p"
-			(at 45.974 86.106 0)
+			(at 46.736 87.376 0)
 			(show_name no)
 			(do_not_autoplace no)
@@
 		)
 		(property "Footprint" "PrLib:C_disc_D7_W2.5_P5"
-			(at 44.7548 80.01 0)
+			(at 47.9552 81.28 0)
 			(hide yes)
 			(show_name no)
@@
 		)
 		(property "Datasheet" ""
-			(at 45.72 83.82 0)
+			(at 46.99 85.09 0)
 			(hide yes)
 			(show_name no)
@@
 		)
 		(property "Description" "Unpolarized capacitor"
-			(at 45.72 83.82 0)
+			(at 46.99 85.09 0)
 			(hide yes)
 			(show_name no)
@@
 		(dnp no)
 		(fields_autoplaced yes)
-		(property "Reference" "Q13"
+		(property "Reference" "Q3"
 			(at 63.5 76.1999 0)
 			(show_name no)
@@
 			(project "AMP-MA"
 				(path "/4094031b-a9da-4ac5-aaa1-42b342c92a3e"
-					(reference "Q13")
+					(reference "Q3")
 					(unit 1)
 				)
@@
 	(symbol
 		(lib_id "Device:C")
-		(at 45.72 41.91 180)
+		(at 46.99 41.91 0)
+		(mirror x)
 		(unit 1)
 		(body_style 1)
@@
 		(dnp no)
 		(property "Reference" "C25"
-			(at 45.974 39.878 0)
+			(at 46.736 39.878 0)
 			(show_name no)
 			(do_not_autoplace no)
@@
 		)
 		(property "Value" "10p"
-			(at 45.974 44.196 0)
+			(at 46.736 44.196 0)
 			(show_name no)
 			(do_not_autoplace no)
@@
 		)
 		(property "Footprint" "PrLib:C_disc_D7_W2.5_P5"
-			(at 44.7548 38.1 0)
+			(at 47.9552 38.1 0)
 			(hide yes)
 			(show_name no)
@@
 		)
 		(property "Datasheet" ""
-			(at 45.72 41.91 0)
+			(at 46.99 41.91 0)
 			(hide yes)
 			(show_name no)
@@
 		)
 		(property "Description" "Unpolarized capacitor"
-			(at 45.72 41.91 0)
+			(at 46.99 41.91 0)
 			(hide yes)
 			(show_name no)
@@
 	(symbol
 		(lib_id "Device:R")
-		(at 40.64 83.82 0)
+		(at 40.64 85.09 0)
 		(unit 1)
 		(body_style 1)
@@
 		(dnp no)
 		(property "Reference" "R15"
-			(at 39.37 82.804 0)
+			(at 39.37 84.074 0)
 			(show_name no)
 			(do_not_autoplace no)
@@
 		)
 		(property "Value" "1M"
-			(at 39.37 85.09 0)
+			(at 39.37 86.36 0)
 			(show_name no)
 			(do_not_autoplace no)
@@
 		)
 		(property "Footprint" "Resistor_THT:R_Axial_DIN0207_L6.3mm_D2.5mm_P10.16mm_Horizontal"
-			(at 38.862 83.82 90)
+			(at 38.862 85.09 90)
 			(hide yes)
 			(show_name no)
@@
 		)
 		(property "Datasheet" ""
-			(at 40.64 83.82 0)
+			(at 40.64 85.09 0)
 			(hide yes)
 			(show_name no)
@@
 		)
 		(property "Description" "Resistor"
-			(at 40.64 83.82 0)
+			(at 40.64 85.09 0)
 			(hide yes)
 			(show_name no)
@@
 		(dnp no)
 		(fields_autoplaced yes)
-		(property "Reference" "Q12"
+		(property "Reference" "Q4"
 			(at 63.5 63.4999 0)
 			(show_name no)
@@
 			(project "AMP-MA"
 				(path "/4094031b-a9da-4ac5-aaa1-42b342c92a3e"
-					(reference "Q12")
+					(reference "Q4")
 					(unit 1)
 				)

Commit message: Revert "Beta 0.0.1"
Parts:
- renumbered Q4 to Q12, Q3 to Q13
Connections:
- net U3_3: no longer names the net of R21.2, R22.2, U3.3 (+)
Other:
- moved on the sheet: C25, C30, R15
Changed lines of the file:
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@@
 	)
 	(junction
-		(at 46.99 36.83)
+		(at 45.72 36.83)
 		(diameter 0)
 		(color 0 0 0 0)
@@
 	)
 	(junction
-		(at 46.99 78.74)
+		(at 45.72 78.74)
 		(diameter 0)
 		(color 0 0 0 0)
@@
 	)
 	(junction
-		(at 46.99 50.8)
+		(at 45.72 50.8)
 		(diameter 0)
 		(color 0 0 0 0)
@@
 	)
 	(junction
-		(at 46.99 92.71)
+		(at 45.72 92.71)
 		(diameter 0)
 		(color 0 0 0 0)
@@
 	(wire
 		(pts
+			(xy 45.72 78.74) (xy 53.34 78.74)
+		)
+		(stroke
+			(width 0)
+			(type default)
+		)
+	)
+	(wire
+		(pts
 			(xy 158.75 67.31) (xy 158.75 73.66)
 		)
@@
 	(wire
 		(pts
+			(xy 54.61 50.8) (xy 45.72 50.8)
+		)
+		(stroke
+			(width 0)
+			(type default)
+		)
+	)
+	(wire
+		(pts
 			(xy 59.69 16.51) (xy 59.69 17.78)
 		)
@@
 	(wire
 		(pts
+			(xy 45.72 36.83) (xy 52.07 36.83)
+		)
+		(stroke
+			(width 0)
+			(type default)
+		)
+	)
+	(wire
+		(pts
 			(xy 29.21 71.12) (xy 29.21 73.66)
 		)
@@
 	(wire
 		(pts
-			(xy 40.64 88.9) (xy 40.64 92.71)
+			(xy 40.64 87.63) (xy 40.64 92.71)
 		)
 		(stroke
@@
 	(wire
 		(pts
-			(xy 46.99 38.1) (xy 46.99 36.83)
+			(xy 45.72 38.1) (xy 45.72 36.83)
 		)
 		(stroke
@@
 	(wire
 		(pts
+			(xy 45.72 92.71) (xy 55.88 92.71)
+		)
+		(stroke
+			(width 0)
+			(type default)
+		)
+	)
+	(wire
+		(pts
 			(xy 118.11 95.25) (xy 120.65 95.25)
 		)
@@
 	(wire
 		(pts
-			(xy 40.64 92.71) (xy 55.88 92.71)
+			(xy 40.64 92.71) (xy 45.72 92.71)
 		)
 		(stroke
@@
 	(wire
 		(pts
-			(xy 46.99 81.28) (xy 46.99 78.74)
+			(xy 45.72 80.01) (xy 45.72 78.74)
 		)
 		(stroke
@@
 	(wire
 		(pts
-			(xy 40.64 78.74) (xy 40.64 81.28)
+			(xy 40.64 78.74) (xy 40.64 80.01)
 		)
 		(stroke
@@
 	(wire
 		(pts
-			(xy 46.99 88.9) (xy 46.99 92.71)
+			(xy 45.72 87.63) (xy 45.72 92.71)
 		)
 		(stroke
@@
 	(wire
 		(pts
-			(xy 46.99 45.72) (xy 46.99 50.8)
+			(xy 45.72 45.72) (xy 45.72 50.8)
 		)
 		(stroke
@@
 	(wire
 		(pts
-			(xy 40.64 78.74) (xy 53.34 78.74)
+			(xy 40.64 78.74) (xy 45.72 78.74)
 		)
 		(stroke
@@
 	(wire
 		(pts
-			(xy 40.64 50.8) (xy 54.61 50.8)
+			(xy 40.64 50.8) (xy 45.72 50.8)
 		)
 		(stroke
@@
 	(wire
 		(pts
-			(xy 40.64 36.83) (xy 52.07 36.83)
+			(xy 40.64 36.83) (xy 45.72 36.83)
 		)
 		(stroke
@@
 		)
 	)
-	(label "U3_3"
-		(at 45.72 111.76 0)
-		(effects
-			(font
-				(size 1.27 1.27)
-			)
-			(justify left bottom)
-		)
-	)
 	(label "LM_IN+"
 		(at 121.92 71.12 0)
@@
 	(symbol
 		(lib_id "Device:C")
-		(at 46.99 85.09 0)
-		(mirror x)
+		(at 45.72 83.82 180)
 		(unit 1)
 		(body_style 1)
@@
 		(dnp no)
 		(property "Reference" "C30"
-			(at 46.736 83.058 0)
+			(at 45.974 81.788 0)
 			(show_name no)
 			(do_not_autoplace no)
@@
 		)
 		(property "Value" "10p"
-			(at 46.736 87.376 0)
+			(at 45.974 86.106 0)
 			(show_name no)
 			(do_not_autoplace no)
@@
 		)
 		(property "Footprint" "PrLib:C_disc_D7_W2.5_P5"
-			(at 47.9552 81.28 0)
+			(at 44.7548 80.01 0)
 			(hide yes)
 			(show_name no)
@@
 		)
 		(property "Datasheet" ""
-			(at 46.99 85.09 0)
+			(at 45.72 83.82 0)
 			(hide yes)
 			(show_name no)
@@
 		)
 		(property "Description" "Unpolarized capacitor"
-			(at 46.99 85.09 0)
+			(at 45.72 83.82 0)
 			(hide yes)
 			(show_name no)
@@
 		(dnp no)
 		(fields_autoplaced yes)
-		(property "Reference" "Q3"
+		(property "Reference" "Q13"
 			(at 63.5 76.1999 0)
 			(show_name no)
@@
 			(project "AMP-MA"
 				(path "/4094031b-a9da-4ac5-aaa1-42b342c92a3e"
-					(reference "Q3")
+					(reference "Q13")
 					(unit 1)
 				)
@@
 	(symbol
 		(lib_id "Device:C")
-		(at 46.99 41.91 0)
-		(mirror x)
+		(at 45.72 41.91 180)
 		(unit 1)
 		(body_style 1)
@@
 		(dnp no)
 		(property "Reference" "C25"
-			(at 46.736 39.878 0)
+			(at 45.974 39.878 0)
 			(show_name no)
 			(do_not_autoplace no)
@@
 		)
 		(property "Value" "10p"
-			(at 46.736 44.196 0)
+			(at 45.974 44.196 0)
 			(show_name no)
 			(do_not_autoplace no)
@@
 		)
 		(property "Footprint" "PrLib:C_disc_D7_W2.5_P5"
-			(at 47.9552 38.1 0)
+			(at 44.7548 38.1 0)
 			(hide yes)
 			(show_name no)
@@
 		)
 		(property "Datasheet" ""
-			(at 46.99 41.91 0)
+			(at 45.72 41.91 0)
 			(hide yes)
 			(show_name no)
@@
 		)
 		(property "Description" "Unpolarized capacitor"
-			(at 46.99 41.91 0)
+			(at 45.72 41.91 0)
 			(hide yes)
 			(show_name no)
@@
 	(symbol
 		(lib_id "Device:R")
-		(at 40.64 85.09 0)
+		(at 40.64 83.82 0)
 		(unit 1)
 		(body_style 1)
@@
 		(dnp no)
 		(property "Reference" "R15"
-			(at 39.37 84.074 0)
+			(at 39.37 82.804 0)
 			(show_name no)
 			(do_not_autoplace no)
@@
 		)
 		(property "Value" "1M"
-			(at 39.37 86.36 0)
+			(at 39.37 85.09 0)
 			(show_name no)
 			(do_not_autoplace no)
@@
 		)
 		(property "Footprint" "Resistor_THT:R_Axial_DIN0207_L6.3mm_D2.5mm_P10.16mm_Horizontal"
-			(at 38.862 85.09 90)
+			(at 38.862 83.82 90)
 			(hide yes)
 			(show_name no)
@@
 		)
 		(property "Datasheet" ""
-			(at 40.64 85.09 0)
+			(at 40.64 83.82 0)
 			(hide yes)
 			(show_name no)
@@
 		)
 		(property "Description" "Resistor"
-			(at 40.64 85.09 0)
+			(at 40.64 83.82 0)
 			(hide yes)
 			(show_name no)
@@
 		(dnp no)
 		(fields_autoplaced yes)
-		(property "Reference" "Q4"
+		(property "Reference" "Q12"
 			(at 63.5 63.4999 0)
 			(show_name no)
@@
 			(project "AMP-MA"
 				(path "/4094031b-a9da-4ac5-aaa1-42b342c92a3e"
-					(reference "Q4")
+					(reference "Q12")
 					(unit 1)
 				)
