File: AMP-MA.kicad_pcb (KiCad board)
At the start: 2 copper layers, 240 x 100 mm, 133 parts, among them J3 Phase, J4 PX Ph, J5 PXB10C, J8 Conn_01x05_Socket, Q1 2N5484, Q10 J201, Q11 J201, Q12 2N5484, Q13 2N5484, Q2 2N5484, Q3 2SC1815, Q4 2SC1815, Q5 2SC1815, Q6 2SC1815, Q7 2SC1815, Q8 2SC1815, SW1 SW_SPDT, U1 CA3080, U3 TL072, U4 LM317_TO-220

Commit message: PCB and Schem upd
Parts:
- added R1: 220R, Resistor_THT:R_Axial_DIN0614_L14.3mm_D5.7mm_P20.32mm_Horizontal, F.Cu at (155.4, 46.9)
- added R2: 220R, Resistor_THT:R_Axial_DIN0614_L14.3mm_D5.7mm_P20.32mm_Horizontal, F.Cu at (155.4, 60.6)
- R39, R46: value 5K -> 4K7
- R54: value 10K -> 4K7
- moved C26 405.8 mm to (40.6, 108.8), turned to 90 degrees
- moved C32 405.1 mm to (88.5, 108.8), turned to 90 degrees
- moved C25 402.7 mm to (44.0, 106.0)
- moved C30 394.3 mm to (97.0, 106.0), turned to 180 degrees
- moved Q1 390.8 mm to (46.5, 101.9)
- moved C29 388.6 mm to (106.1, 121.3), turned to 90 degrees
- moved C24 388.4 mm to (58.0, 121.3), turned to 90 degrees
- moved Q13 387.3 mm to (92.7, 101.9)
- moved R38 384.1 mm to (33.4, 103.8), turned to -90 degrees
- moved R7 382.5 mm to (36.9, 103.8), turned to -90 degrees
- moved C33 382.4 mm to (114.4, 126.7), turned to -90 degrees
- moved C28 382.3 mm to (66.4, 126.6), turned to -90 degrees
- moved R45 382.0 mm to (81.2, 103.8), turned to -90 degrees
- moved C31 374.4 mm to (124.6, 126.6), turned to 180 degrees
- moved R44 374.1 mm to (85.0, 103.8), turned to -90 degrees
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Connections:
- net /Compression block/PREAMP renamed PREAMP
- C1 pad 1: /power supply/VCC -> VCC
- C10 pad 2: /Compression block/VB -> VB
- C18 pad 1: /power supply/VEE -> VEE
- C19 pad 1: /power supply/VCC -> VCC
- C2 pad 1: /CP_OUT -> CP_OUT
- C34 pad 1: /VEE -> VEE
- C6 pad 2: /VCC -> VCC
- C9 pad 2: /Compression block/VB -> VB
- CE1 pad 1: /power supply/VC -> VC
- CE2 pad 1: /power supply/VCC -> VCC
- CE3 pad 2: /power supply/VEE -> VEE
- CE4 pad 1: /power supply/VB -> VB
- CE5 pad 1: /power supply/VMu -> VMu
- CE6 pad 1: /VCC -> VCC
- CE7 pad 2: /VEE -> VEE
- D10 pad 2: /power supply/VEE -> VEE
- D5 pad 2: /power supply/VB -> VB
- D7 pad 2: /power supply/VEE -> VEE
- D8 pad 1: /power supply/VCC -> VCC
- D9 pad 1: /power supply/VCC -> VCC
- J8 pad 3: /VEE -> VEE
- J8 pad 4: /VCC -> VCC
- Q10 pad 2: /Compression block/OUTPUT -> CP_OUT
- Q11 pad 2: /Compression block/OUTPUT -> CP_OUT
- Q12 pad 1: /VMu -> VMu
- Q2 pad 1: /VMu -> VMu
- Q6 pad 2: /Compression block/VC -> VC
- R12 pad 2: /Compression block/VC -> VC
- R14 pad 2: /Compression block/VB -> VB
- R17 pad 1: /Compression block/VC -> VC
- R19 pad 2: /Compression block/VC -> VC
- R22 pad 1: /Compression block/VC -> VC
- R25 pad 1: /Compression block/VC -> VC
- R29 pad 1: /power supply/VC -> VC
- R3 pad 1: /power supply/VC -> VC
- R3 pad 2: /power supply/VB -> VB
- R33 pad 1: /Compression block/VB -> VB
- R34 pad 1: /Compression block/VB -> VB
- R34 pad 2: /Compression block/OUTPUT -> CP_OUT
- R35 pad 1: /Compression block/VB -> VB
- R4 pad 1: /power supply/VB -> VB
- R41 pad 1: /VMu -> VMu
- R48 pad 2: /CP_OUT -> CP_OUT
- R5 pad 1: /power supply/VMu -> VMu
- R5 pad 2: /power supply/VC -> VC
- R9 pad 1: /VMu -> VMu
- U3 pad 5: (no net) -> unconnected-(U3B-+-Pad5)
- U3 pad 6: (no net) -> unconnected-(U3B---Pad6)
- U3 pad 7: (no net) -> unconnected-(U3-Pad7)
- U4 pad 2: /power supply/VC -> VC
- U4 pad 3: /power supply/VCC -> VCC
Routing:
- net Net-(Q12-S): track 0.00 -> 49.5 mm
- net Net-(Q1-D): track 0.00 -> 49.5 mm
- net VCC: track 0.00 -> 48.0 mm
- net VEE: track 0.00 -> 44.7 mm
- net Net-(Q13-G): track 0.00 -> 26.7 mm
- net Net-(D10-K): track 0.00 -> 23.9 mm
- net Net-(Q1-G): track 0.00 -> 18.2 mm
- net Net-(Q1-S): track 0.00 -> 16.0 mm
- net Net-(Q2-G): track 0.00 -> 15.0 mm
- net Net-(Q12-G): track 0.00 -> 14.9 mm
- net Net-(Q13-S): track 0.00 -> 13.9 mm, vias 0 -> 1
- net Net-(D7-K): track 0.00 -> 13.8 mm
- net VMu: track 0.00 -> 13.6 mm
- net Net-(C24-Pad1): track 0.00 -> 5.17 mm
- net Net-(C29-Pad1): track 0.00 -> 5.10 mm
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- added copper zone on B.Cu, net GND
- added copper zone on F.Cu, net GND

Commit message: Big upd
fully routed pcb. Some small updates for Schematic
Parts:
- removed the R20 at (324.8, 117.7)
- removed the R21 at (324.8, 121.7)
- removed R27: 800R, Resistor_THT:R_Axial_DIN0207_L6.3mm_D2.5mm_P10.16mm_Horizontal
- removed the R53 at (353.0, 99.5)
- added J9: Socket_01x03, Connector_JST:JST_XH_B3B-XH-A_1x03_P2.50mm_Vertical, F.Cu at (264.2, 104.2)
- added R40: 20K, Resistor_THT:R_Axial_DIN0207_L6.3mm_D2.5mm_P10.16mm_Horizontal, F.Cu at (140.0, 76.4)
- added R47: 800R, Resistor_THT:R_Axial_DIN0207_L6.3mm_D2.5mm_P10.16mm_Horizontal, F.Cu at (266.0, 126.9)
- C1, C10, C11, C12, C13, C14, C15, C16, C17, C18, C19, C2, C20, C21, C22, C23, C24, C25, C26, C27, C28, C29, C3, C30, C31, C32, C33, C34, C35, C36, C4, C5, C6, C7, C8, C9: footprint Capacitor_THT:C_Disc_D7.0mm_W2.5mm_P5.00mm -> PrLib:C_disc_D7_W2.5_P5
- J3, J4: footprint Connector_Phoenix_SPT:PhoenixContact_SPT_2.5_1-H-5.0_1x01_P5.0mm_Horizontal -> PrLib:connector
- J5: footprint Connector_JST:JST_PH_B3B-PH-K_1x03_P2.00mm_Vertical -> Connector_JST:JST_XH_B3B-XH-A_1x03_P2.50mm_Vertical
- J8: value Conn_01x05_Socket -> Socket_01x05; footprint Connector_JST:JST_PH_B5B-PH-K_1x05_P2.00mm_Vertical -> Connector_JST:JST_XH_B5B-XH-A_1x05_P2.50mm_Vertical
- RBass1, RMiddle1, RTreble1, VOL1, VOL2: footprint Potentiometer_THT:Potentiometer_Alps_RK09Y11_Single_Horizontal -> PrLib:potentiometer
- SW1: value SW_SPDT -> SW_DPDT_x2; footprint Button_Switch_THT:SW_CK_JS202011AQN_DPDT_Angled -> PrLib:SW DPDT
- moved CE8 334.6 mm to (47.5, 58.9), turned to 180 degrees
- moved R61 303.4 mm to (51.4, 58.9)
- moved C5 301.1 mm to (66.3, 55.4), turned to 90 degrees
- moved CE6 294.1 mm to (88.9, 46.3), turned to 90 degrees
- moved R62 293.3 mm to (61.5, 54.6), turned to 90 degrees
- moved C34 291.9 mm to (93.3, 48.8), turned to -90 degrees
- moved C6 285.2 mm to (83.1, 51.3), turned to 90 degrees
- moved CE7 283.8 mm to (98.8, 46.3), turned to -90 degrees
- moved R64 275.7 mm to (79.3, 50.4), turned to 180 degrees
- moved R63 274.3 mm to (79.4, 55.4), turned to 180 degrees
- moved U1 251.4 mm to (118.3, 57.8)
- moved RV1 246.4 mm to (112.2, 62.8), turned to 180 degrees
- moved R30 223.3 mm to (95.3, 57.8), turned to -90 degrees
- moved C2 222.7 mm to (151.5, 125.0), turned to 180 degrees
- moved C8 216.1 mm to (107.1, 76.5), turned to 180 degrees
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- renumbered R6 to R10, R7 to R11, R38 to R12, R8 to R13, R9 to R14, R40 to R15, R44 to R16, R45 to R17, R42 to R18, R41 to R19, R54 to R20, R46 to R21, R39 to R22, R11 to R30, R12 to R31, R10 to R32, R13 to R33, R14 to R34, R15 to R35, R17 to R36, R16 to R37, R18 to R38, R19 to R39, R25 to R41, R22 to R42, R24 to R43, R23 to R44, R28 to R45, R32 to R46, R34 to R50, R36 to R51, R37 to R52, R35 to R53, R33 to R54, R48 to R55, R30 to R6, R52 to R60, R51 to R61, R50 to R62, R47 to R63, R49 to R64, R29 to R7
Connections:
- C14 pad 1: unconnected-(C14-Pad1) -> Net-(Q8-B)
- C15 pad 1: Net-(SW1-C) -> Net-(SW1A-C)
- C16 pad 1: Net-(SW1-A) -> Net-(SW1A-A)
- C17 pad 1: Net-(Q8-C) -> /Compression block/BP_OUT
- C17 pad 2: unconnected-(C17-Pad2) -> Net-(Q7-B)
- C21 pad 1: /Compression block/PREAMP_OUT -> PREAMP
- D5 pad 2: VB -> /Compression block/BP_OUT
- LS1 pad 1: GND -> Net-(J9-Pin_3)
- Q8 pad 2: Net-(Q8-C) -> /Compression block/BP_OUT
- R20 pad 2: /PREAMP -> PREAMP
- R41 pad 2: Net-(Q8-C) -> /Compression block/BP_OUT
- R45 pad 2: Net-(SW1-B) -> Net-(SW1A-B)
- SW1 pad 1: Net-(SW1-A) -> Net-(SW1A-A)
- SW1 pad 2: Net-(SW1-B) -> Net-(SW1A-B)
- SW1 pad 3: Net-(SW1-C) -> Net-(SW1A-C)
- SW1 pad 4: (no net) -> Net-(SW1A-A)
- SW1 pad 5: (no net) -> Net-(SW1A-B)
- SW1 pad 6: (no net) -> Net-(SW1A-C)
- U1 pad 4: /Compression block/VEE -> VEE
- U1 pad 7: /Compression block/VCC -> VCC
- U3 pad 1: /PREAMP -> PREAMP
Routing:
- net VC: track 0.00 -> 255.6 mm
- net /LM_OUT: track 0.00 -> 245.4 mm
- net PREAMP: track 0.00 -> 212.0 mm, vias 0 -> 1
- net GND: track 236.1 -> 39.2 mm
- net VCC: track 48.0 -> 238.0 mm
- net VEE: track 44.7 -> 213.9 mm
- net VB: track 0.00 -> 149.9 mm
- net /ToneSt: track 0.00 -> 134.8 mm
- net /Compression block/CP_IN: track 0.00 -> 124.6 mm
- net CP_OUT: track 0.00 -> 99.8 mm
- net /Compression block/BP_OUT: track 0.00 -> 85.2 mm
- net VMu: track 13.6 -> 94.1 mm
- net Net-(U3A-+): track 0.00 -> 51.0 mm
- net /Compression block/EFF_OUT: track 0.00 -> 48.1 mm
- net Net-(Q3-B): track 0.00 -> 44.6 mm, vias 0 -> 1
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- added copper zone on B.Cu, net (none)
- added copper zone on F.Cu, net (none)
Other:
- outline, holes or cut-outs redrawn

Commit message: small upd
changed & added capacitor footprint. replaced potentimeters
Parts:
- C10, C11, C12, C14, C15, C16, C17, C22, C23, C9: footprint PrLib:C_disc_D7_W2.5_P5 -> PrLib:C_Disc_D4.3_W1.9_P5.00
- LEVEL: renamed from LEVEL1; footprint Potentiometer_THT:Potentiometer_Alps_RK09Y11_Single_Horizontal -> PrLib:potentiometer
- R62: value 20K -> 22K
- moved Q10 10.1 mm to (226.5, 126.5)
- moved C23 7.95 mm to (226.5, 116.8)
- moved Q11 3.98 mm to (231.3, 116.2)
- moved C14 3.46 mm to (214.1, 101.5)
- moved LEVEL 2.82 mm to (236.0, 136.0), turned to 0 degrees
- moved C36 2.75 mm to (248.0, 134.7)
- moved R50 2.39 mm to (241.2, 119.9)
- moved R43 2.19 mm to (207.1, 118.0)
- moved R44 2.19 mm to (202.0, 118.0)
- moved R41 1.95 mm to (226.0, 112.5)
- moved C22 1.90 mm to (240.2, 116.2)
- moved C20 1.75 mm to (231.0, 126.5)
- moved Bass 1.30 mm to (198.0, 136.0)
- moved Middle 1.30 mm to (174.0, 136.0)
- moved VOL1 1.30 mm to (78.0, 136.0)
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- renumbered RBass1 to Bass, RMiddle1 to Middle, RTreble1 to Treble
Routing:
- net Net-(Q10-G): track 18.3 -> 8.47 mm
- net Net-(Q10-D): track 14.0 -> 7.75 mm
- net Net-(Q7-B): track 26.7 -> 31.3 mm
- net Net-(Q11-G): track 14.1 -> 9.90 mm
- net Net-(C20-Pad2): track 6.45 -> 9.50 mm
- net /Compression block/CP_IN: track 124.6 -> 127.4 mm
- net VC: track 255.6 -> 258.3 mm
- net Net-(Q8-B): track 38.9 -> 41.2 mm
- net CP_OUT: track 99.8 -> 98.0 mm
- net /Compression block/BP_OUT: track 85.2 -> 87.0 mm
- net /Compression block/EFF_OUT: track 48.1 -> 49.7 mm
- net /ToneSt: track 134.8 -> 136.1 mm
- net /PREAMP1: track 27.8 -> 29.1 mm
- net VB: track 149.9 -> 151.2 mm
- net Net-(C28-Pad2): track 9.77 -> 11.0 mm
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Other:
- board text added: "100KA"
- board text added: "220KA"
- board text added: "22KA"

Commit message: First Beta
Parts:
- added GND: MountingHole_Pad, MountingHole:MountingHole_2.2mm_M2_DIN965_Pad, F.Cu at (145.0, 55.0)
- added H1: MountingHole, MountingHole:MountingHole_2.2mm_M2, F.Cu at (70.0, 45.0)
- added H2: MountingHole, MountingHole:MountingHole_2.2mm_M2, F.Cu at (214.0, 45.0)
- RV1, RV2: footprint Potentiometer_THT:Potentiometer_ACP_CA9-H2,5_Horizontal -> Potentiometer_THT:Potentiometer_Bourns_3296W_Vertical
- moved J2 1.07 mm to (101.7, 128.7)
- moved C2 0.75 mm to (151.5, 124.2)
- moved C26 0.30 mm to (47.7, 108.5)
- moved R11 0.30 mm to (44.1, 103.5)
- moved R12 0.30 mm to (40.5, 103.5)
- moved C24 0.30 mm to (65.2, 121.0)
- moved C25 0.30 mm to (51.2, 105.7)
- moved Q1 0.30 mm to (53.6, 101.6)
- moved R10 0.30 mm to (61.1, 110.7)
- moved J1 0.22 mm to (50.6, 128.7)
- moved J8 0.10 mm to (53.2, 53.8)
- moved CE6 0.07 mm to (88.9, 46.3)
- moved C6 0.06 mm to (83.2, 51.3)
- turned RV1 to -90 degrees
- turned RV2 to -90 degrees
Routing:
- net GND: track 39.2 -> 0.04 mm
- net VC: track 258.3 -> 253.7 mm
- net /LM_OUT: track 245.4 -> 242.3 mm
- net /Compression block/BP_OUT: track 87.0 -> 84.1 mm
- net Net-(Q12-S): track 49.8 -> 46.9 mm
- net Net-(Q1-D): track 49.9 -> 47.0 mm
- net PREAMP: track 212.5 -> 210.1 mm
- net Net-(R31-Pad1): track 6.13 -> 8.55 mm
- net /ToneSt: track 136.1 -> 133.7 mm
- net Net-(R40-Pad1): track 43.8 -> 41.6 mm
- net /Compression block/CP_IN: track 127.4 -> 125.2 mm
- net VB: track 151.2 -> 149.2 mm
- net VMu: track 93.8 -> 91.9 mm
- net CP_OUT: track 98.0 -> 96.4 mm
- net Net-(Bass1-Pad3): track 37.7 -> 36.4 mm
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Other:
- outline, holes or cut-outs redrawn

Commit message: Patch 0
PCB updates
Parts:
- moved C19 9.97 mm to (42.7, 84.6), turned to 0 degrees
- moved R1 5.85 mm to (106.0, 92.6)
- moved C18 5.58 mm to (106.0, 86.9), turned to 0 degrees
- moved R2 2.47 mm to (42.7, 90.5)
- moved F1 1.85 mm to (225.6, 69.0)
- moved J3 1.85 mm to (225.6, 75.2)
- moved J4 1.85 mm to (225.6, 43.8)
- moved C36 1.30 mm to (248.0, 136.0)
- moved R20 0.26 mm to (57.1, 95.4)
Routing:
- net Net-(J3-Pin_1): track 17.0 -> 34.1 mm
- net Net-(J4-Pin_1): track 15.5 -> 31.0 mm
- net VCC: track 237.9 -> 233.9 mm
- net Net-(U3C-V-): track 8.87 -> 5.63 mm
- net Net-(U3C-V+): track 9.62 -> 10.4 mm
- net GND: vias 0 -> 27
Other:
- board text added: "100KB"
- board text added: "220V"

Commit message: Patch 1
Major PCB update
Parts:
- moved Q8 13.1 mm to (210.6, 97.2), turned to -90 degrees
- moved C17 12.8 mm to (206.4, 98.5)
- moved C14 7.71 mm to (206.4, 101.0), turned to 180 degrees
- moved Q7 6.73 mm to (199.1, 101.0)
- moved R30 6.54 mm to (101.8, 57.8)
- moved C8 4.96 mm to (112.0, 76.5)
- moved R63 4.21 mm to (78.5, 59.6)
- moved C5 4.21 mm to (65.5, 59.6)
- moved R64 3.75 mm to (75.7, 51.3)
- moved R42 3.61 mm to (226.0, 101.0)
- moved R31 2.61 mm to (106.3, 60.3)
- moved R46 1.30 mm to (184.9, 114.7)
- moved D6 1.30 mm to (184.9, 101.0)
- moved C35 1.25 mm to (253.0, 107.1)
- moved J9 1.25 mm to (263.0, 104.2)
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Routing:
- net Net-(Q8-B): track 40.2 -> 24.9 mm
- net Net-(D6-A): track 12.8 -> 25.9 mm
- net /Compression block/BP_OUT: track 84.1 -> 78.2 mm
- net Net-(C7-Pad2): track 11.9 -> 6.97 mm
- net /Compression block/EFF_OUT: track 48.8 -> 53.3 mm
- net /ToneSt: track 133.7 -> 129.9 mm, vias 0 -> 1
- net Net-(Q7-B): track 30.8 -> 27.7 mm
- net Net-(R31-Pad1): track 8.55 -> 5.94 mm
- net /LM_OUT: track 242.3 -> 240.7 mm
- net Net-(Q1-G): track 18.0 -> 19.4 mm
- net VC: track 253.7 -> 255.0 mm
- net Net-(Q13-G): track 18.4 -> 19.6 mm
- net Net-(C33-Pad2): track 10.9 -> 11.9 mm
- net Net-(C28-Pad2): track 11.0 -> 11.9 mm
- net /PREAMP2: track 29.1 -> 29.9 mm
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Other:
- board size 240 x 100 mm -> 230 x 100 mm
