File: AMP-MA.kicad_pcb (KiCad board)
At the start: 2 copper layers, 230 x 100 mm, 137 parts, among them J3 Phase, J4 PX Ph, J5 PXB10C, J8 Socket_01x05, J9 Socket_01x03, Q1 2N5484, Q10 J201, Q11 J201, Q12 2N5484, Q13 2N5484, Q2 2N5484, Q3 2SC1815, Q4 2SC1815, Q5 2SC1815, Q6 2SC1815, Q7 2SC1815, Q8 2SC1815, SW1 SW_DPDT_x2, U1 CA3080, U3 TL072, U4 LM317_TO-220

Commit message: Patch 2 gitignore update
PCB update
Parts:
- added G***: LOGO, LOGO, F.Cu at (89.4, 68.8)

Commit message: Repository cleaned up
Parts:
- moved C19 0.24 mm to (42.7, 84.8)
Routing:
- net /PREAMP1: track 29.9 -> 30.9 mm
- net /PREAMP2: track 29.9 -> 30.9 mm

Commit message: PCB upd
Traces upd, created net classes
Parts:
- moved C18 0.75 mm to (106.0, 86.2)
- moved R42 0.23 mm to (225.8, 101.1)
- moved R41 0.22 mm to (225.8, 112.5)
- moved C21 0.18 mm to (223.7, 108.0)
- moved R53 0.18 mm to (238.8, 111.3)
- moved R51 0.07 mm to (241.6, 111.3)
Routing:
- net /Compression block/EFF_OUT: track 53.3 -> 52.4 mm
- net VB: track 149.2 -> 149.7 mm
- net VC: track 255.0 -> 254.8 mm, vias 0 -> 1
- net GND: vias 48 -> 38
