File: AMP-MA.kicad_pcb (KiCad board)
At the start: 2 copper layers, 230 x 100 mm, 138 parts, among them J3 Phase, J4 PX Ph, J5 PXB10C, J8 Socket_01x05, J9 Socket_01x03, Q1 2N5484, Q10 J201, Q11 J201, Q12 2N5484, Q13 2N5484, Q2 2N5484, Q3 2SC1815, Q4 2SC1815, Q5 2SC1815, Q6 2SC1815, Q7 2SC1815, Q8 2SC1815, SW1 SW_DPDT_x2, U1 CA3080, U3 TL072, U4 LM317_TO-220

Commit message: Version 0.1.0 Pre-Release
Reworked PCB, reanotated some components, changed some footprints
Parts:
- removed Bass, Treble: 220KA, PrLib:potentiometer
- removed the C10 at (132.8, 66.1)
- removed the C14 at (206.4, 101.0)
- removed the C16 at (207.1, 123.5)
- removed the C17 at (206.4, 98.5)
- removed the C19 at (42.7, 84.8)
- removed the C2 at (152.4, 124.2)
- removed C22, C23: 10n, PrLib:C_Disc_D4.3_W1.9_P5.00
- removed C29: 50n, PrLib:C_disc_D7_W2.5_P5
- removed C3, C4: 22n, PrLib:C_disc_D7_W2.5_P5
- removed C36: 100n, PrLib:C_disc_D7_W2.5_P5
- removed J3: Phase, PrLib:connector
- removed J4: PX Ph, PrLib:connector
- removed J9: Socket_01x03, Connector_JST:JST_XH_B3B-XH-A_1x03_P2.50mm_Vertical
- removed LEVEL: 100KB, PrLib:potentiometer
- removed Middle: 22KA, PrLib:potentiometer
- removed Q12, Q13: 2N5484, Package_TO_SOT_THT:TO-92_Inline
- removed the Q7 at (199.1, 101.0)
- removed the Q8 at (210.6, 97.2)
- removed the R1 at (106.0, 92.6)
- removed the R2 at (42.7, 90.5)
- removed the R41 at (226.0, 112.5)
- removed R46: 100R, Resistor_THT:R_Axial_DIN0207_L6.3mm_D2.5mm_P10.16mm_Horizontal
- removed R54: 510K, Resistor_THT:R_Axial_DIN0207_L6.3mm_D2.5mm_P10.16mm_Horizontal
- removed R55: 33K, Resistor_THT:R_Axial_DIN0207_L6.3mm_D2.5mm_P10.16mm_Horizontal
- added Bass1: Bass, PrLib:potentiometer, F.Cu at (152.0, 142.0)
- added C41: 100n, PrLib:C_disc_D7_W2.5_P5, F.Cu at (170.5, 122.5)
- added C42: 10n, PrLib:C_Disc_D4.3_W1.9_P5.00, F.Cu at (179.9, 120.2)
- added C43: 10n, PrLib:C_Disc_D4.3_W1.9_P5.00, F.Cu at (182.9, 102.7)
- added C44: 100n, PrLib:C_disc_D7_W2.5_P5, F.Cu at (175.4, 119.0)
- added C45: 100n, PrLib:C_disc_D7_W2.5_P5, F.Cu at (170.4, 103.2)
- added C51: C51, PrLib:C_disc_D7_W2.5_P5, F.Cu at (198.0, 130.4)
- added C52: C52, PrLib:C_disc_D7_W2.5_P5, F.Cu at (152.0, 125.5)
- added C53: C53, PrLib:C_disc_D7_W2.5_P5, F.Cu at (171.0, 125.5)
- added C54: C54, PrLib:C_disc_D7_W2.5_P5, F.Cu at (157.0, 133.6)
- added C55: C55, PrLib:C_disc_D7_W2.5_P5, F.Cu at (190.0, 133.6)
- added C56: C56, PrLib:C_disc_D7_W2.5_P5, F.Cu at (196.1, 117.9)
- added CE4: 100u, Capacitor_THT:CP_Radial_D6.3mm_P2.50mm, F.Cu at (180.3, 78.5)
- added CE5: 10u, Capacitor_THT:CP_Radial_D6.3mm_P2.50mm, F.Cu at (160.7, 69.0)
- added CE6: 10u, Capacitor_THT:CP_Radial_D6.3mm_P2.50mm, F.Cu at (160.7, 91.6)
- added D0: LED, LED_THT:LED_D3.0mm_Horizontal_O6.35mm_Z6.0mm, F.Cu at (252.7, 141.4)
- added D10: 1N4001, Diode_THT:D_DO-41_SOD81_P10.16mm_Horizontal, F.Cu at (174.6, 85.4)
- added D7: 1N4001, Diode_THT:D_DO-41_SOD81_P10.16mm_Horizontal, F.Cu at (163.8, 75.3)
- added D8: 1N4001, Diode_THT:D_DO-41_SOD81_P10.16mm_Horizontal, F.Cu at (167.6, 85.4)
- added D9: 1N4001, Diode_THT:D_DO-41_SOD81_P10.16mm_Horizontal, F.Cu at (174.0, 57.7)
- added J1: Neutral, PrLib:connector, F.Cu at (227.6, 81.3)
- added J2: PXB N, PrLib:connector, F.Cu at (227.6, 49.8)
- added JP0: SolderJumper_2_Open, Jumper:SolderJumper-2_P1.3mm_Open_TrianglePad1.0x1.5mm, F.Cu at (200.0, 117.2)
- added JP50: SolderJumper_3_Open, Jumper:SolderJumper-3_P2.0mm_Open_TrianglePad1.0x1.5mm_NumberLabels, F.Cu at (193.0, 127.4)
- added JP51: SolderJumper_3_Open, Jumper:SolderJumper-3_P2.0mm_Open_TrianglePad1.0x1.5mm_NumberLabels, F.Cu at (173.0, 133.5)
- added JP52: SolderJumper_2_Open, Jumper:SolderJumper-2_P1.3mm_Open_TrianglePad1.0x1.5mm, F.Cu at (164.0, 142.0)
- added LEVEL1: 100KB, Potentiometer_THT:Potentiometer_Bourns_3296W_Vertical, F.Cu at (160.9, 122.5)
- added Middle1: Middle, PrLib:potentiometer, F.Cu at (176.0, 142.0)
- added OUT2: External Speaker, Connector_JST:JST_XH_B3B-XH-A_1x03_P2.50mm_Vertical, F.Cu at (265.0, 110.3)
- added Q3: 2SK30A, Package_TO_SOT_THT:TO-92_Inline_Wide, F.Cu at (111.4, 109.3)
- added Q4: 2SK30A, Package_TO_SOT_THT:TO-92_Inline_Wide, F.Cu at (117.5, 117.8)
- added R23: 1K5, Resistor_THT:R_Axial_DIN0207_L6.3mm_D2.5mm_P10.16mm_Horizontal, F.Cu at (131.2, 105.3)
- added R24: 1K5, Resistor_THT:R_Axial_DIN0207_L6.3mm_D2.5mm_P10.16mm_Horizontal, F.Cu at (134.3, 95.0)
- added R3: 200R, Resistor_THT:R_Axial_DIN0207_L6.3mm_D2.5mm_P10.16mm_Horizontal, F.Cu at (171.1, 75.2)
- added R4: 2K2, Resistor_THT:R_Axial_DIN0207_L6.3mm_D2.5mm_P10.16mm_Horizontal, F.Cu at (160.6, 85.4)
- added R50: Rin, Resistor_THT:R_Axial_DIN0207_L6.3mm_D2.5mm_P10.16mm_Horizontal, F.Cu at (206.0, 133.1)
- added RV50: 1M, Potentiometer_THT:Potentiometer_Bourns_3296W_Vertical, F.Cu at (191.5, 117.9)
- added Treble1: Treble, PrLib:potentiometer, F.Cu at (200.0, 142.0)
- added U5: LM337_TO220, Package_TO_SOT_THT:TO-220-3_Horizontal_TabDown, F.Cu at (160.6, 80.3)
- C13: renamed from C28; value 220n -> 330n
- C15: value 1n -> 50n; footprint PrLib:C_Disc_D4.3_W1.9_P5.00 -> PrLib:C_disc_D7_W2.5_P5
- C18: renamed from C33; value 220n -> 330n
- C20, C21: value 100n -> 1u
- C31: renamed from C9; value 1n -> 2n2
- C35: renamed from C13; footprint PrLib:C_disc_D7_W2.5_P5 -> Capacitor_THT:CP_Radial_Tantal_D5.5mm_P2.50mm
- C61: renamed from C6; value 0.1u -> 100n
- C62: renamed from C34; value 0.1u -> 100n
- C8: value 1u/10 -> 1u
- CE1: renamed from CE2; footprint Capacitor_THT:CP_Radial_D14.0mm_P7.50mm -> Capacitor_THT:CP_Radial_D16.0mm_P7.50mm
- CE2: renamed from CE3; footprint Capacitor_THT:CP_Radial_D14.0mm_P7.50mm -> Capacitor_THT:CP_Radial_D16.0mm_P7.50mm
- D31: renamed from D1; value 1N914 -> 1N4148
- D32: renamed from D3; value 1N914 -> 1N4148
- D5: value LED -> 1N4001; footprint LED_THT:LED_D3.0mm_Horizontal_O6.35mm_Z6.0mm -> Diode_THT:D_DO-41_SOD81_P10.16mm_Horizontal
- D6: value 1N914 -> 1N4001; footprint Diode_THT:D_DO-35_SOD27_P7.62mm_Horizontal -> Diode_THT:D_DO-41_SOD81_P10.16mm_Horizontal
- F1: moved to B.Cu
- J6: renamed from J8; value Socket_01x05 -> LM1875
- Q1, Q2: value 2N5484 -> 2SK30A; footprint Package_TO_SOT_THT:TO-92_Inline -> Package_TO_SOT_THT:TO-92_Inline_Wide
- Q10, Q11: value J201 -> 2SK30A; footprint Package_TO_SOT_THT:TO-92_Inline -> Package_TO_SOT_THT:TO-92_Inline_Wide
- Q5: renamed from Q4; footprint Package_TO_SOT_THT:TO-92_Inline -> Package_TO_SOT_THT:TO-92_Inline_Wide
- Q6: renamed from Q5; footprint Package_TO_SOT_THT:TO-92_Inline -> Package_TO_SOT_THT:TO-92_Inline_Wide
- Q7: renamed from Q6; footprint Package_TO_SOT_THT:TO-92_Inline -> Package_TO_SOT_THT:TO-92_Inline_Wide
- Q8: renamed from Q3; footprint Package_TO_SOT_THT:TO-92_Inline -> Package_TO_SOT_THT:TO-92_Inline_Wide
- R0: renamed from R47; value 800R -> 1K5
- R1: renamed from R7; value 240R -> 200R
- R10, R15: value 1M -> 2M
- R2: renamed from R6; value 2K -> 2K2
- R20: value 4K7 -> 50K
- R21: renamed from R22; value 4K7 -> 100K
- R22: renamed from R21; value 4K7 -> 100K
- R42: value 10K -> 1M
- R43: value 56K -> 1M
- R44: value 56K -> 510K
- R45: value 22R -> 510K
- R5: renamed from R3; footprint Resistor_THT:R_Axial_DIN0207_L6.3mm_D2.5mm_P7.62mm_Horizontal -> Resistor_THT:R_Axial_DIN0207_L6.3mm_D2.5mm_P10.16mm_Horizontal
- R51: value 1M -> R51
- R52: value 1M -> R52
- R53: value 510K -> R53
- R6: renamed from R4; footprint Resistor_THT:R_Axial_DIN0207_L6.3mm_D2.5mm_P7.62mm_Horizontal -> Resistor_THT:R_Axial_DIN0207_L6.3mm_D2.5mm_P10.16mm_Horizontal
- R60: value 1R -> 2R2
- R7: renamed from R5; footprint Resistor_THT:R_Axial_DIN0207_L6.3mm_D2.5mm_P7.62mm_Horizontal -> Resistor_THT:R_Axial_DIN0207_L6.3mm_D2.5mm_P10.16mm_Horizontal
- Sustain1: renamed from RV2; footprint Potentiometer_THT:Potentiometer_Bourns_3296W_Vertical -> PrLib:potentiometer
- U4: value LM317_TO-220 -> LM317
- moved C20 161.2 mm to (70.0, 133.8)
- moved D5 128.8 mm to (163.7, 47.9), turned to -90 degrees
- moved R40 124.2 mm to (248.2, 137.2), turned to 0 degrees
- moved R30 113.9 mm to (209.4, 95.0)
- moved C21 108.6 mm to (118.0, 133.8)
- moved U3 101.4 mm to (212.3, 95.6)
- moved R31 100.5 mm to (199.7, 97.5), turned to -90 degrees
- moved RV1 99.7 mm to (204.7, 100.1)
- moved R33 98.2 mm to (216.0, 110.0)
- moved R32 98.0 mm to (203.0, 117.3), turned to 0 degrees
- moved C30 97.9 mm to (210.8, 113.2)
- moved C8 97.9 mm to (202.8, 113.2), turned to 90 degrees
- moved C31 97.2 mm to (222.3, 100.7)
- moved R34 95.9 mm to (222.3, 104.0)
- moved Q5 86.8 mm to (245.0, 128.3), turned to 90 degrees
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- renumbered C24 to C10, C25 to C11, C26 to C12, C27 to C14, C30 to C16, C32 to C17, C31 to C19, C18 to C2, C7 to C30, C12 to C33, C11 to C34, C35 to C60, C5 to C63, CE1 to CE3, CE6 to CE61, CE7 to CE62, CE8 to CE63, CE5 to CE7, CE4 to CE8, D8 to D1, D9 to D2, D7 to D3, D10 to D4, GND to GND1, J1 to IN1, J2 to IN2, LS1 to OUT1, R50 to R41, U3 to U1, U1 to U3
Connections:
- net /ToneSt renamed TS_OUT
- C13 pad 2: Net-(C28-Pad2) -> Net-(C13-Pad2)
- C15 pad 1: Net-(SW1A-C) -> Net-(C15-Pad1)
- C15 pad 2: Net-(Q7-B) -> Net-(Q3-G)
- C16 pad 2: Net-(Q13-G) -> Net-(Q3-G)
- C18 pad 2: Net-(C33-Pad2) -> Net-(C18-Pad2)
- C20 pad 1: Net-(Q10-D) -> GND
- C21 pad 1: PREAMP -> GND
- C21 pad 2: Net-(Q11-D) -> Net-(C21-Pad2)
- D1 pad 2: Net-(D7-K) -> PXB_3
- D2 pad 2: Net-(D10-K) -> PXB_1
- D3 pad 1: Net-(D7-K) -> PXB_3
- D4 pad 1: Net-(D10-K) -> PXB_1
- D5 pad 1: Net-(D5-K) -> VCC
- D5 pad 2: /Compression block/BP_OUT -> VC
- D6 pad 1: Net-(D6-K) -> VC
- F1 pad 1: Net-(J3-Pin_1) -> Neutral
- F1 pad 2: Net-(J4-Pin_1) -> PXB_N
- IN2 pad T: Net-(C29-Pad1) -> Net-(C15-Pad1)
- J5 pad 1: Net-(D7-K) -> PXB_1
- J5 pad 3: Net-(D10-K) -> PXB_3
- OUT1 pad 1: Net-(J9-Pin_3) -> /Ex_Speaker
- Q1 pad 2: Net-(Q1-S) -> Net-(Q1-G)
- Q1 pad 3: Net-(Q1-G) -> Net-(Q1-S)
- Q10 pad 1: Net-(Q10-D) -> BP_OUT
- Q10 pad 2: CP_OUT -> /Compression block/Q11_3
- Q10 pad 3: Net-(Q10-G) -> Net-(Q10-S)
- Q11 pad 1: Net-(Q11-D) -> BP_OUT
- Q11 pad 2: CP_OUT -> /Compression block/Q10_3
- Q11 pad 3: Net-(Q11-G) -> Net-(Q11-S)
- Q2 pad 2: Net-(Q1-D) -> Net-(Q2-G)
- Q2 pad 3: Net-(Q2-G) -> Net-(Q1-D)
- R0 pad 2: Net-(D5-K) -> Net-(D0-K)
- R1 pad 2: Net-(U4-ADJ) -> Net-(D6-A)
- R15 pad 1: Net-(Q13-G) -> Net-(Q3-G)
- R2 pad 1: Net-(U4-ADJ) -> Net-(D6-A)
- R20 pad 1: GND -> /U3_3
- R20 pad 2: PREAMP -> Net-(R20-Pad2)
- R21 pad 2: Net-(U3A-+) -> /U3_3
- R22 pad 2: Net-(U3A-+) -> /U3_3
- R40 pad 1: Net-(R40-Pad1) -> /Compression block/BIAS
- R40 pad 2: /Compression block/BIAS -> Net-(R40-Pad2)
- R41 pad 2: CP_OUT -> BP_OUT
- R42 pad 1: VC -> /Compression block/Q11_3
- R42 pad 2: /Compression block/EFF_OUT -> /Compression block/ON
- R43 pad 1: Net-(Q8-B) (its old number) -> /Compression block/Q10_3
- R43 pad 2: GND -> /Compression block/OFF
- R44 pad 1: Net-(Q7-B) -> VB
- R44 pad 2: GND -> Net-(Q10-S)
- R45 pad 1: GND -> VB
- R45 pad 2: Net-(SW1A-B) -> Net-(Q11-S)
- R51 pad 1: Net-(Q11-G) -> Net-(C52-Pad1)
- R51 pad 2: /Compression block/EFF_OUT -> Net-(C51-Pad1)
- R52 pad 1: Net-(Q10-G) -> GND
- R52 pad 2: /Compression block/BP_OUT -> Net-(JP52-B)
- R53 pad 1: VB -> GND
- R53 pad 2: Net-(Q11-D) -> Net-(JP50-A)
- SW1 pad 1: Net-(SW1A-A) -> /Compression block/OFF
- SW1 pad 2: Net-(SW1A-B) -> GND
- SW1 pad 3: Net-(SW1A-C) -> /Compression block/ON
- SW1 pad 4: Net-(SW1A-A) -> /Compression block/ON
- SW1 pad 5: Net-(SW1A-B) -> VC
- SW1 pad 6: Net-(SW1A-C) -> /Compression block/OFF
- Sustain1 pad 3: Net-(R40-Pad1) -> Net-(R40-Pad2)
- U1 pad 1: PREAMP -> Net-(R20-Pad2)
- U1 pad 2: GND -> /U3_3
- U1 pad 3: Net-(U3A-+) -> GND
- U1 pad 4: Net-(U3C-V-) -> VE
- U1 pad 5: unconnected-(U3B-+-Pad5) -> GND
- U1 pad 6: unconnected-(U3B---Pad6) -> Net-(U1B--)
- U1 pad 7: unconnected-(U3-Pad7) -> PREAMP
- U1 pad 8: Net-(U3C-V+) -> VC
- U3 pad 4: VEE -> VE
- U3 pad 7: VCC -> VC
- U4 pad 1: Net-(U4-ADJ) -> Net-(D6-A)
- VOL1 pad 1: Net-(C28-Pad2) -> Net-(C20-Pad2)
- VOL1 pad 3: GND -> Net-(C13-Pad2)
- VOL2 pad 1: Net-(C33-Pad2) -> Net-(C21-Pad2)
- VOL2 pad 3: GND -> Net-(C18-Pad2)
Routing:
- net PREAMP: track 209.7 -> 88.4 mm
- net VE: track 0.00 -> 116.2 mm, vias 0 -> 1
- net CP_OUT: track 96.0 -> 0.00 mm
- net /Compression block/ON: track 0.00 -> 83.6 mm, vias 0 -> 2
- net /Compression block/BP_OUT: track 78.2 -> 0.00 mm
- net VCC: track 233.8 -> 156.7 mm
- net /Tone Stack/Bass: track 0.00 -> 70.9 mm
- net /Compression block/CP_IN: track 124.7 -> 57.6 mm, vias 0 -> 1
- net /Compression block/OFF: track 0.00 -> 64.1 mm, vias 0 -> 3
- net /U3_3: track 0.00 -> 60.4 mm
- net /Compression block/EFF_OUT: track 53.3 -> 0.00 mm
- net Net-(C52-Pad1): track 0.00 -> 51.2 mm
- net Net-(U3A-+): track 51.0 -> 0.00 mm
- net BP_OUT: track 0.00 -> 47.4 mm, vias 0 -> 1
- net Net-(Bass1-Pad1): track 44.6 -> 0.00 mm
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Other:
- board size 230 x 100 mm -> 228 x 100 mm
- board text added: "LM337"
- board text removed: "100KB"
- board text removed: "220KA"
- board text removed: "22KA"

Commit message: Version 0.1.0 Release
Parts:
- removed JP0: SolderJumper_2_Open, Jumper:SolderJumper-2_P1.3mm_Open_TrianglePad1.0x1.5mm
- added JP54: SolderJumper_2_Open, Jumper:SolderJumper-2_P1.3mm_Open_TrianglePad1.0x1.5mm, F.Cu at (200.0, 117.2)
- U5: value LM337_TO220 -> LM337
- renumbered Bass1 to Bass, Middle1 to Middle, Sustain1 to Sustain, Treble1 to Treble
Routing:
- net GND: vias 400 -> 378
Other:
- outline, holes or cut-outs redrawn
- board text removed: "100KA"

Commit message: feat: start version 0.2.0 development
Parts:
- removed JP54: SolderJumper_2_Open, Jumper:SolderJumper-2_P1.3mm_Open_TrianglePad1.0x1.5mm
- added J7: LM1875, Connector_JST:JST_XH_B5B-XH-A_1x05_P2.50mm_Vertical, F.Cu at (247.0, 91.0)
- added R54: 1R, Resistor_THT:R_Axial_DIN0207_L6.3mm_D2.5mm_P10.16mm_Horizontal, F.Cu at (200.0, 107.7)
- added U2: LM1875, Package_TO_SOT_THT:TO-220-5_P3.4x3.7mm_StaggerOdd_Lead3.8mm_Vertical, F.Cu at (248.6, 60.2)
- moved R63 195.6 mm to (252.4, 85.5), turned to 180 degrees
- moved CE63 192.1 mm to (241.5, 70.5), turned to -90 degrees
- moved R62 189.8 mm to (252.5, 80.0), turned to 0 degrees
- moved R61 188.1 mm to (241.5, 66.7), turned to 90 degrees
- moved C61 183.7 mm to (260.4, 64.0), turned to 180 degrees
- moved R64 179.1 mm to (245.8, 67.3)
- moved C63 175.3 mm to (242.2, 82.5)
- moved C62 174.9 mm to (252.0, 64.0), turned to 180 degrees
- moved CE61 173.8 mm to (255.4, 69.0), turned to 0 degrees
- moved CE62 163.1 mm to (249.5, 72.5), turned to 0 degrees
- moved J6 63.4 mm to (117.5, 50.5), turned to 0 degrees
- moved G*** 20.1 mm to (86.0, 64.0)
- moved GND1 8.21 mm to (134.0, 57.7)
- moved RV50 5.08 mm to (191.5, 112.8), turned to 90 degrees
- moved C53 3.00 mm to (174.0, 125.5)
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- renumbered Bass to Bass1, Middle to Middle1, Sustain to Sustain1, Treble to Treble1
Connections:
- C56 pad 1: Net-(JP54-A) -> Net-(C56-Pad1)
- C61 pad 1: GND -> GND1
- C61 pad 2: VCC -> /VCC1
- C62 pad 1: VEE -> /VEE1
- C62 pad 2: GND -> GND1
- C63 pad 1: TS_OUT -> /LM_IN
- CE61 pad 1: VCC -> /VCC1
- CE61 pad 2: GND -> GND1
- CE62 pad 1: GND -> GND1
- CE62 pad 2: VEE -> /VEE1
- CE63 pad 2: GND -> GND1
- J6 pad 1: /LM_IN- -> TS_OUT
- J6 pad 2: /LM_IN+ -> /Speaker
- J6 pad 3: VEE -> GND
- J6 pad 4: VCC -> VEE
- J6 pad 5: /LM_OUT -> VCC
- OUT1 pad 2: /LM_OUT -> /Speaker
- OUT2 pad 1: /LM_OUT -> /Speaker
- R60 pad 1: /LM_OUT -> /Speaker
- R63 pad 1: GND -> GND1
- R63 pad 2: TS_OUT -> /LM_IN
- R64 pad 1: GND -> GND1
- RV50 pad 1: Net-(JP54-A) -> GND
- RV50 pad 3: GND -> Net-(C56-Pad1)
- Treble1 pad 2: Net-(JP54-A) -> Net-(C56-Pad1)
Routing:
- net /Speaker: track 0.00 -> 187.3 mm
- net /LM_OUT: track 234.4 -> 55.9 mm
- net VCC: track 156.7 -> 83.3 mm
- net VEE: track 175.4 -> 112.3 mm
- net Net-(C56-Pad1): track 0.00 -> 32.5 mm
- net Net-(JP54-A): track 32.5 -> 0.00 mm
- net /VEE1: track 0.00 -> 31.8 mm
- net /VCC1: track 0.00 -> 31.4 mm
- net /LM_IN-: track 13.3 -> 44.6 mm
- net TS_OUT: track 154.0 -> 126.5 mm
- net /LM_IN: track 0.00 -> 10.3 mm
- net /LM_IN+: track 15.5 -> 21.9 mm
- net VC: track 282.3 -> 284.6 mm
- net Net-(D8-K): track 20.6 -> 22.5 mm
- net /Tone Stack/Mid: track 17.8 -> 19.0 mm
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- added copper zone on B.Cu, net GND1
- added copper zone on F.Cu, net GND1
Other:
- outline, holes or cut-outs redrawn
- board text removed: "2 1 3 5 4"
