File: Schematics/PwSup.kicad_sch (KiCad schematic)
At the start: 30 parts, among them J3 Phase, J4 PX Ph, J5 PXB10C, J6 Neutral, J7 Px N, SW2 SW_SPST, U3 TL072, U4 LM317_TO-220

Commit message: PCB and Schem upd
Parts:
- R1, R2: footprint (none) -> Resistor_THT:R_Axial_DIN0614_L14.3mm_D5.7mm_P20.32mm_Horizontal
Changed lines of the file:
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@@
 	(rectangle
 		(start 72.39 15.24)
-		(end 181.61 58.42)
+		(end 175.895 58.42)
 		(radius 4.064)
 		(stroke
@@
 	)
 	(rectangle
-		(start 151.13 19.05)
-		(end 175.26 43.18)
+		(start 151.13 17.145)
+		(end 172.085 43.18)
 		(stroke
 			(width 0)
@@
 	)
 	(rectangle
-		(start 128.27 19.05)
+		(start 128.27 17.145)
 		(end 149.86 38.1)
 		(stroke
@@
 	(text "block Mu"
 		(exclude_from_sim no)
-		(at 136.144 21.844 0)
+		(at 136.144 20.574 0)
 		(effects
 			(font
@@
 	(text "block B"
 		(exclude_from_sim no)
-		(at 172.974 25.654 90)
+		(at 162.56 20.574 0)
 		(effects
 			(font
@@
 	)
 	(junction
+		(at 160.02 26.67)
+		(diameter 0)
+		(color 0 0 0 0)
+	)
+	(junction
 		(at 105.41 93.98)
 		(diameter 0)
@@
 		(color 0 0 0 0)
 	)
-	(junction
-		(at 160.02 26.67)
-		(diameter 0)
-		(color 0 0 0 0)
-	)
 	(wire
 		(pts
@@
 	(wire
 		(pts
-			(xy 153.67 26.67) (xy 160.02 26.67)
+			(xy 116.84 85.09) (xy 116.84 87.63)
 		)
 		(stroke
@@
 	(wire
 		(pts
-			(xy 116.84 85.09) (xy 116.84 87.63)
+			(xy 55.88 85.09) (xy 62.23 85.09)
 		)
 		(stroke
@@
 	(wire
 		(pts
-			(xy 55.88 85.09) (xy 62.23 85.09)
+			(xy 160.02 26.67) (xy 160.02 39.37)
 		)
 		(stroke
@@
 	(wire
 		(pts
-			(xy 160.02 39.37) (xy 160.02 26.67)
+			(xy 60.96 87.63) (xy 55.88 87.63)
 		)
 		(stroke
@@
 	(wire
 		(pts
-			(xy 60.96 87.63) (xy 55.88 87.63)
+			(xy 38.1 80.01) (xy 36.83 80.01)
 		)
 		(stroke
@@
 	(wire
 		(pts
-			(xy 38.1 80.01) (xy 36.83 80.01)
+			(xy 60.96 73.66) (xy 60.96 82.55)
 		)
 		(stroke
@@
 	(wire
 		(pts
-			(xy 60.96 73.66) (xy 60.96 82.55)
+			(xy 105.41 82.55) (xy 105.41 76.2)
 		)
 		(stroke
@@
 	(wire
 		(pts
-			(xy 105.41 82.55) (xy 105.41 76.2)
+			(xy 146.05 24.13) (xy 146.05 27.94)
 		)
 		(stroke
@@
 	(wire
 		(pts
-			(xy 146.05 20.32) (xy 146.05 27.94)
+			(xy 125.73 39.37) (xy 125.73 43.18)
 		)
 		(stroke
@@
 	(wire
 		(pts
-			(xy 125.73 39.37) (xy 125.73 43.18)
+			(xy 157.48 26.67) (xy 160.02 26.67)
 		)
 		(stroke
@@
 		)
 	)
-	(label "VC"
-		(at 125.73 33.02 270)
+	(label "VCC"
+		(at 54.61 55.88 0)
 		(effects
 			(font
 				(size 1.27 1.27)
 			)
-			(justify right bottom)
+			(justify left bottom)
 		)
 	)
-	(label "VB"
-		(at 146.05 52.07 0)
+	(label "VCC"
+		(at 76.2 39.37 0)
 		(effects
 			(font
@@
 		)
 	)
-	(label "VCC"
-		(at 76.2 39.37 0)
+	(label "VEE"
+		(at 66.04 55.88 0)
 		(effects
 			(font
@@
 		)
 	)
-	(label "VB"
-		(at 153.67 26.67 0)
+	(label "VCC"
+		(at 102.87 76.2 180)
 		(effects
 			(font
 				(size 1.27 1.27)
 			)
-			(justify left bottom)
+			(justify right bottom)
 		)
 	)
-	(label "VCC"
-		(at 102.87 76.2 180)
+	(global_label "VB"
+		(shape input)
+		(at 146.05 52.07 180)
+		(fields_autoplaced yes)
 		(effects
 			(font
 				(size 1.27 1.27)
 			)
-			(justify right bottom)
+			(justify right)
+		)
+		(property "Intersheetrefs" "${INTERSHEET_REFS}"
+			(at 140.7062 52.07 0)
+			(hide yes)
+			(show_name no)
+			(do_not_autoplace no)
+			(effects
+				(font
+					(size 1.27 1.27)
+				)
+				(justify right)
+			)
 		)
 	)
-	(label "VMu"
-		(at 146.05 20.32 270)
+	(global_label "VB"
+		(shape input)
+		(at 157.48 26.67 180)
+		(fields_autoplaced yes)
 		(effects
 			(font
 				(size 1.27 1.27)
 			)
-			(justify right bottom)
+			(justify right)
+		)
+		(property "Intersheetrefs" "${INTERSHEET_REFS}"
+			(at 152.1362 26.67 0)
+			(hide yes)
+			(show_name no)
+			(do_not_autoplace no)
+			(effects
+				(font
+					(size 1.27 1.27)
+				)
+				(justify right)
+			)
+		)
+	)
+	(global_label "VEE"
+		(shape input)
+		(at 66.04 55.88 180)
+		(fields_autoplaced yes)
+		(effects
+			(font
+				(size 1.27 1.27)
+			)
+			(justify right)
+		)
+		(property "Intersheetrefs" "${INTERSHEET_REFS}"
+			(at 59.6682 55.88 0)
+			(hide yes)
+			(show_name no)
+			(do_not_autoplace no)
+			(effects
+				(font
+					(size 1.27 1.27)
+				)
+				(justify right)
+			)
+		)
+	)
+	(global_label "VMu"
+		(shape input)
+		(at 146.05 24.13 90)
+		(fields_autoplaced yes)
+		(effects
+			(font
+				(size 1.27 1.27)
+			)
+			(justify left)
+		)
+		(property "Intersheetrefs" "${INTERSHEET_REFS}"
+			(at 146.05 17.4558 90)
+			(hide yes)
+			(show_name no)
+			(do_not_autoplace no)
+			(effects
+				(font
+					(size 1.27 1.27)
+				)
+				(justify left)
+			)
+		)
+	)
+	(global_label "VCC"
+		(shape input)
+		(at 54.61 55.88 180)
+		(fields_autoplaced yes)
+		(effects
+			(font
+				(size 1.27 1.27)
+			)
+			(justify right)
+		)
+		(property "Intersheetrefs" "${INTERSHEET_REFS}"
+			(at 47.9962 55.88 0)
+			(hide yes)
+			(show_name no)
+			(do_not_autoplace no)
+			(effects
+				(font
+					(size 1.27 1.27)
+				)
+				(justify right)
+			)
+		)
+	)
+	(global_label "VC"
+		(shape input)
+		(at 125.73 33.02 90)
+		(fields_autoplaced yes)
+		(effects
+			(font
+				(size 1.27 1.27)
+			)
+			(justify left)
+		)
+		(property "Intersheetrefs" "${INTERSHEET_REFS}"
+			(at 125.73 27.6762 90)
+			(hide yes)
+			(show_name no)
+			(do_not_autoplace no)
+			(effects
+				(font
+					(size 1.27 1.27)
+				)
+				(justify left)
+			)
 		)
 	)
@@
 			)
 		)
-		(property "Footprint" ""
+		(property "Footprint" "Resistor_THT:R_Axial_DIN0614_L14.3mm_D5.7mm_P20.32mm_Horizontal"
 			(at 110.49 77.978 90)
 			(hide yes)
@@
 			)
 		)
-		(property "Footprint" ""
+		(property "Footprint" "Resistor_THT:R_Axial_DIN0614_L14.3mm_D5.7mm_P20.32mm_Horizontal"
 			(at 110.49 95.758 90)
 			(hide yes)

Commit message: Big upd
fully routed pcb. Some small updates for Schematic
Parts:
- removed D5: LED, LED_THT:LED_D3.0mm_Horizontal_O6.35mm_Z6.0mm, symbol Device:LED
- removed R27: 800R, Resistor_THT:R_Axial_DIN0207_L6.3mm_D2.5mm_P10.16mm_Horizontal, symbol Device:R
- C1, C18, C19: footprint Capacitor_THT:C_Disc_D7.0mm_W2.5mm_P5.00mm -> PrLib:C_disc_D7_W2.5_P5
- J3, J4: footprint Connector_Phoenix_SPT:PhoenixContact_SPT_2.5_1-H-5.0_1x01_P5.0mm_Horizontal -> PrLib:connector
- J5: footprint Connector_JST:JST_PH_B3B-PH-K_1x03_P2.00mm_Vertical -> Connector_JST:JST_XH_B3B-XH-A_1x03_P2.50mm_Vertical
- renumbered R30 to R6, R29 to R7
