File: Schematics/PwSup.kicad_sch (KiCad schematic)
At the start: 28 parts, among them J3 Neutral, J4 Px N, J5 PXB10C, J6 Phase, J7 Px Ph, SW2 SW_SPST, U3 TL072, U4 LM317_TO-220

Commit message: Revert "Beta 0.0.1"
Parts:
- J3: value Neutral -> Phase
- J4: value Px N -> PX Ph
- J6: value Phase -> Neutral
- J7: value Px Ph -> Px N
Other:
- moved on the sheet: C18, C19, CE2, CE3, D10, D7, D8, D9, F1, J3, J4, J5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
