File: Schematics/Cp.kicad_sch (KiCad schematic)
At the start: 55 parts, among them Q10 J201, Q11 J201, Q3 2SC1815, Q4 2SC1815, Q5 2SC1815, Q6 2SC1815, Q7 2SC1815, Q8 2SC1815, SW1 SW_SPDT, U1 CA3080

Commit message: PCB and Schem upd
Connections:
- net OUTPUT renamed CP_OUT
Other:
- moved on the sheet: C14, C15, C16, C17, D6, Q7, Q8, R22, R23, R24, R25, R28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

Commit message: Big upd
fully routed pcb. Some small updates for Schematic
Parts:
- removed R21: 10K, Resistor_THT:R_Axial_DIN0207_L6.3mm_D2.5mm_P10.16mm_Horizontal, symbol Device:R
- removed SW1: SW_SPDT, Button_Switch_THT:SW_CK_JS202011AQN_DPDT_Angled, symbol Switch:SW_SPDT
- added D5: LED, LED_THT:LED_D3.0mm_Horizontal_O6.35mm_Z6.0mm, symbol Device:LED
- added R47: 800R, Resistor_THT:R_Axial_DIN0207_L6.3mm_D2.5mm_P10.16mm_Horizontal, symbol Device:R
- added SW1: SW_DPDT_x2, PrLib:SW DPDT, symbol Switch:SW_DPDT_x2
- C10, C11, C12, C13, C14, C15, C16, C17, C20, C21, C22, C23, C36, C7, C8, C9: footprint Capacitor_THT:C_Disc_D7.0mm_W2.5mm_P5.00mm -> PrLib:C_disc_D7_W2.5_P5
- R40: renamed from R20; value 10K -> 20K
- renumbered R11 to R30, R12 to R31, R10 to R32, R13 to R33, R14 to R34, R15 to R35, R17 to R36, R16 to R37, R18 to R38, R19 to R39, R25 to R41, R22 to R42, R24 to R43, R23 to R44, R28 to R45, R32 to R46, R34 to R50, R36 to R51, R37 to R52, R35 to R53, R33 to R54
Connections:
- net PREAMP_OUT is gone; now on net PREAMP: C21.1
- net BIAS: now also R40.2
- net BP_OUT: now also C17.1, Q8.2 (C), R41.2, D5.2 (A)
- net GND: now also R47.1
- net at C17.2: now also C15.2, Q7.3 (B), R44.1
- net at C16.2, Q8.3 (B), R43.1: now also C14.1
- net at C15.1: now also SW1.3 (C), SW1.6 (C)
- net at C16.1: now also SW1.1 (A), SW1.4 (A)
- net at R45.2: now also SW1.2 (B), SW1.5 (B)
- new net: D5.1 (K), R47.2
Other:
- moved on the sheet: C14, C15, C16, C17, D6, Q7, Q8, R41, R42, R43, R44, R45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

Commit message: small upd
changed & added capacitor footprint. replaced potentimeters
Parts:
- C10, C11, C12, C14, C15, C16, C17, C22, C23, C9: footprint PrLib:C_disc_D7_W2.5_P5 -> PrLib:C_Disc_D4.3_W1.9_P5.00
- LEVEL1: footprint Potentiometer_THT:Potentiometer_Alps_RK09Y11_Single_Horizontal -> PrLib:potentiometer
Changed lines of the file:
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@@
 			)
 		)
-		(property "Footprint" "PrLib:C_disc_D7_W2.5_P5"
+		(property "Footprint" "PrLib:C_Disc_D4.3_W1.9_P5.00"
 			(at 77.1652 46.99 0)
 			(hide yes)
@@
 			)
 		)
-		(property "Footprint" "PrLib:C_disc_D7_W2.5_P5"
+		(property "Footprint" "PrLib:C_Disc_D4.3_W1.9_P5.00"
 			(at 110.49 44.7548 0)
 			(hide yes)
@@
 			)
 		)
-		(property "Footprint" "Potentiometer_THT:Potentiometer_Alps_RK09Y11_Single_Horizontal"
+		(property "Footprint" "PrLib:potentiometer"
 			(at 154.94 91.44 0)
 			(hide yes)
@@
 			)
 		)
-		(property "Footprint" "PrLib:C_disc_D7_W2.5_P5"
+		(property "Footprint" "PrLib:C_Disc_D4.3_W1.9_P5.00"
 			(at 57.15 84.1248 0)
 			(hide yes)
@@
 			)
 		)
-		(property "Footprint" "PrLib:C_disc_D7_W2.5_P5"
+		(property "Footprint" "PrLib:C_Disc_D4.3_W1.9_P5.00"
 			(at 76.2 84.1248 0)
 			(hide yes)
@@
 			)
 		)
-		(property "Footprint" "PrLib:C_disc_D7_W2.5_P5"
+		(property "Footprint" "PrLib:C_Disc_D4.3_W1.9_P5.00"
 			(at 120.3452 105.41 0)
 			(hide yes)
@@
 			)
 		)
-		(property "Footprint" "PrLib:C_disc_D7_W2.5_P5"
+		(property "Footprint" "PrLib:C_Disc_D4.3_W1.9_P5.00"
 			(at 110.49 29.5148 0)
 			(hide yes)
@@
 			)
 		)
-		(property "Footprint" "PrLib:C_disc_D7_W2.5_P5"
+		(property "Footprint" "PrLib:C_Disc_D4.3_W1.9_P5.00"
 			(at 70.1548 46.99 0)
 			(hide yes)
@@
 			)
 		)
-		(property "Footprint" "PrLib:C_disc_D7_W2.5_P5"
+		(property "Footprint" "PrLib:C_Disc_D4.3_W1.9_P5.00"
 			(at 69.5452 92.71 0)
 			(hide yes)
@@
 			)
 		)
-		(property "Footprint" "PrLib:C_disc_D7_W2.5_P5"
+		(property "Footprint" "PrLib:C_Disc_D4.3_W1.9_P5.00"
 			(at 57.4548 92.71 0)
 			(hide yes)
@@
 			)
 		)
-		(property "Footprint" "PrLib:C_disc_D7_W2.5_P5"
+		(property "Footprint" "PrLib:C_Disc_D4.3_W1.9_P5.00"
 			(at 126.0348 105.41 0)
 			(hide yes)

Commit message: First Beta
Parts:
- R47: value 800R -> 1K5
- RV1, RV2: footprint Potentiometer_THT:Potentiometer_ACP_CA9-H2,5_Horizontal -> Potentiometer_THT:Potentiometer_Bourns_3296W_Vertical
Changed lines of the file:
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@@
 			)
 		)
-		(property "Footprint" "Potentiometer_THT:Potentiometer_ACP_CA9-H2,5_Horizontal"
+		(property "Footprint" "Potentiometer_THT:Potentiometer_Bourns_3296W_Vertical"
 			(at 36.83 40.64 0)
 			(hide yes)
@@
 			)
 		)
-		(property "Footprint" "Potentiometer_THT:Potentiometer_ACP_CA9-H2,5_Horizontal"
+		(property "Footprint" "Potentiometer_THT:Potentiometer_Bourns_3296W_Vertical"
 			(at 160.02 53.34 0)
 			(hide yes)
@@
 			)
 		)
-		(property "Value" "800R"
-			(at 26.67 82.804 90)
+		(property "Value" "1K5"
+			(at 26.162 82.804 90)
 			(show_name no)
 			(do_not_autoplace no)

Commit message: Dev(#4)
* Patch 0

PCB updates

* Patch 1

Major PCB update

* Delete AMP-MA-backups directory

* Patch 2 gitignore update

PCB update

* Repository cleaned up

* PCB upd

Traces upd, created net classes

* Beta Version 0.0.1

Traces upd, Readme Upd
Parts:
- renumbered Q11 to Q10, Q10 to Q11, Q4 to Q5, Q5 to Q6, Q6 to Q7, Q7 to Q9
Connections:
- net SW_A: now reaches C16.1, SW1.1 (A), SW1.4 (A)
- net SW_C: now reaches C15.1, SW1.3 (C), SW1.6 (C)
- net Q9_3: now reaches C15.2, C17.2, Q9.3 (B), R44.1
- net Q8_3: now reaches C14.1, C16.2, Q8.3 (B), R43.1
- net Q10_3: now reaches C22.2, Q10.3 (G), R51.1
- net Q11_3: now reaches C23.2, Q11.3 (G), R52.1
Changed lines of the file:
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@@
 	(wire
 		(pts
-			(xy 58.42 101.6) (xy 60.96 101.6)
-		)
-		(stroke
-			(width 0)
-			(type default)
-		)
-	)
-	(wire
-		(pts
 			(xy 71.12 39.37) (xy 71.12 38.1)
 		)
@@
 	(wire
 		(pts
+			(xy 58.42 101.6) (xy 60.96 101.6)
+		)
+		(stroke
+			(width 0)
+			(type default)
+		)
+	)
+	(wire
+		(pts
 			(xy 82.55 46.99) (xy 82.55 48.26)
 		)
@@
 	(wire
 		(pts
-			(xy 68.58 100.33) (xy 68.58 101.6)
-		)
-		(stroke
-			(width 0)
-			(type default)
-		)
-	)
-	(wire
-		(pts
 			(xy 27.94 80.01) (xy 36.83 80.01)
 		)
@@
 	(wire
 		(pts
-			(xy 58.42 101.6) (xy 58.42 100.33)
-		)
-		(stroke
-			(width 0)
-			(type default)
-		)
-	)
-	(wire
-		(pts
 			(xy 110.49 30.48) (xy 113.03 30.48)
 		)
@@
 	(wire
 		(pts
+			(xy 68.58 101.6) (xy 68.58 100.33)
+		)
+		(stroke
+			(width 0)
+			(type default)
+		)
+	)
+	(wire
+		(pts
 			(xy 132.08 24.13) (xy 139.7 24.13)
 		)
@@
 	(wire
 		(pts
+			(xy 58.42 101.6) (xy 58.42 100.33)
+		)
+		(stroke
+			(width 0)
+			(type default)
+		)
+	)
+	(wire
+		(pts
 			(xy 41.91 83.82) (xy 41.91 85.09)
 		)
@@
 		)
 	)
+	(label "Q10_3"
+		(at 118.11 104.14 180)
+		(effects
+			(font
+				(size 1.27 1.27)
+			)
+			(justify right bottom)
+		)
+	)
 	(label "BIAS"
 		(at 160.02 38.1 270)
@@
 		)
 	)
+	(label "SW_C"
+		(at 68.58 101.6 180)
+		(effects
+			(font
+				(size 1.27 1.27)
+			)
+			(justify right bottom)
+		)
+	)
+	(label "Q9_3"
+		(at 76.2 92.71 180)
+		(effects
+			(font
+				(size 1.27 1.27)
+			)
+			(justify right bottom)
+		)
+	)
 	(label "VC"
 		(at 96.52 17.78 270)
@@
 		)
 	)
+	(label "Q8_3"
+		(at 50.8 91.44 0)
+		(effects
+			(font
+				(size 1.27 1.27)
+			)
+			(justify left bottom)
+		)
+	)
 	(label "BP_OUT"
 		(at 133.35 121.92 90)
@@
 		)
 	)
+	(label "Q11_3"
+		(at 128.27 104.14 0)
+		(effects
+			(font
+				(size 1.27 1.27)
+			)
+			(justify left bottom)
+		)
+	)
+	(label "SW_A"
+		(at 58.42 101.6 0)
+		(effects
+			(font
+				(size 1.27 1.27)
+			)
+			(justify left bottom)
+		)
+	)
 	(global_label "VC"
 		(shape input)
@@
 		(in_pos_files yes)
 		(dnp no)
-		(property "Reference" "Q5"
+		(property "Reference" "Q6"
 			(at 127 34.29 0)
 			(show_name no)
@@
 			(project "AMP-MA"
 				(path "/4094031b-a9da-4ac5-aaa1-42b342c92a3e/d432553b-ab0c-45ec-bbdd-5af2e9267855"
-					(reference "Q5")
+					(reference "Q6")
 					(unit 1)
 				)
@@
 		(in_pos_files yes)
 		(dnp no)
-		(property "Reference" "Q11"
+		(property "Reference" "Q10"
 			(at 116.84 89.154 90)
 			(show_name no)
@@
 			(project "AMP-MA"
 				(path "/4094031b-a9da-4ac5-aaa1-42b342c92a3e/d432553b-ab0c-45ec-bbdd-5af2e9267855"
-					(reference "Q11")
+					(reference "Q10")
 					(unit 1)
 				)
@@
 		(in_pos_files yes)
 		(dnp no)
-		(property "Reference" "Q6"
+		(property "Reference" "Q7"
 			(at 150.622 34.036 0)
 			(show_name no)
@@
 			(project "AMP-MA"
 				(path "/4094031b-a9da-4ac5-aaa1-42b342c92a3e/d432553b-ab0c-45ec-bbdd-5af2e9267855"
-					(reference "Q6")
+					(reference "Q7")
 					(unit 1)
 				)
@@
 		(in_pos_files yes)
 		(dnp no)
-		(property "Reference" "Q10"
+		(property "Reference" "Q11"
 			(at 129.54 89.408 90)
 			(show_name no)
@@
 			(project "AMP-MA"
 				(path "/4094031b-a9da-4ac5-aaa1-42b342c92a3e/d432553b-ab0c-45ec-bbdd-5af2e9267855"
-					(reference "Q10")
+					(reference "Q11")
 					(unit 1)
 				)
@@
 		(in_pos_files yes)
 		(dnp no)
-		(property "Reference" "Q7"
+		(property "Reference" "Q9"
 			(at 80.518 88.646 0)
 			(show_name no)
@@
 			(project "AMP-MA"
 				(path "/4094031b-a9da-4ac5-aaa1-42b342c92a3e/d432553b-ab0c-45ec-bbdd-5af2e9267855"
-					(reference "Q7")
+					(reference "Q9")
 					(unit 1)
 				)
@@
 		(in_pos_files yes)
 		(dnp no)
-		(property "Reference" "Q4"
+		(property "Reference" "Q5"
 			(at 127 42.164 0)
 			(show_name no)
@@
 			(project "AMP-MA"
 				(path "/4094031b-a9da-4ac5-aaa1-42b342c92a3e/d432553b-ab0c-45ec-bbdd-5af2e9267855"
-					(reference "Q4")
+					(reference "Q5")
 					(unit 1)
 				)

Commit message: Revert "Beta 0.0.1"
Parts:
- renumbered Q11 to Q10, Q10 to Q11, Q5 to Q4, Q6 to Q5, Q7 to Q6, Q9 to Q7
Connections:
- net Q10_3: no longer names the net of C22.2, Q11.3 (G), R51.1
- net Q11_3: no longer names the net of C23.2, Q10.3 (G), R52.1
- net Q8_3: no longer names the net of C14.1, C16.2, Q8.3 (B), R43.1
- net Q9_3: no longer names the net of C15.2, C17.2, Q7.3 (B), R44.1
- net SW_A: no longer names the net of C16.1, SW1.1 (A), SW1.4 (A)
- net SW_C: no longer names the net of C15.1, SW1.3 (C), SW1.6 (C)
Changed lines of the file:
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@@
 	(wire
 		(pts
+			(xy 58.42 101.6) (xy 60.96 101.6)
+		)
+		(stroke
+			(width 0)
+			(type default)
+		)
+	)
+	(wire
+		(pts
 			(xy 71.12 39.37) (xy 71.12 38.1)
 		)
@@
 	(wire
 		(pts
-			(xy 58.42 101.6) (xy 60.96 101.6)
-		)
-		(stroke
-			(width 0)
-			(type default)
-		)
-	)
-	(wire
-		(pts
 			(xy 82.55 46.99) (xy 82.55 48.26)
 		)
@@
 	(wire
 		(pts
+			(xy 68.58 100.33) (xy 68.58 101.6)
+		)
+		(stroke
+			(width 0)
+			(type default)
+		)
+	)
+	(wire
+		(pts
 			(xy 27.94 80.01) (xy 36.83 80.01)
 		)
@@
 	(wire
 		(pts
-			(xy 110.49 30.48) (xy 113.03 30.48)
+			(xy 58.42 101.6) (xy 58.42 100.33)
 		)
 		(stroke
@@
 	(wire
 		(pts
-			(xy 124.46 45.72) (xy 123.19 45.72)
+			(xy 110.49 30.48) (xy 113.03 30.48)
 		)
 		(stroke
@@
 	(wire
 		(pts
-			(xy 27.94 35.56) (xy 29.21 35.56)
+			(xy 124.46 45.72) (xy 123.19 45.72)
 		)
 		(stroke
@@
 	(wire
 		(pts
-			(xy 68.58 92.71) (xy 76.2 92.71)
+			(xy 27.94 35.56) (xy 29.21 35.56)
 		)
 		(stroke
@@
 	(wire
 		(pts
-			(xy 123.19 82.55) (xy 123.19 78.74)
+			(xy 68.58 92.71) (xy 76.2 92.71)
 		)
 		(stroke
@@
 	(wire
 		(pts
-			(xy 132.08 52.07) (xy 132.08 50.8)
+			(xy 123.19 82.55) (xy 123.19 78.74)
 		)
 		(stroke
@@
 	(wire
 		(pts
-			(xy 76.2 48.26) (xy 76.2 46.99)
+			(xy 132.08 52.07) (xy 132.08 50.8)
 		)
 		(stroke
@@
 	(wire
 		(pts
-			(xy 142.24 38.1) (xy 139.7 38.1)
+			(xy 76.2 48.26) (xy 76.2 46.99)
 		)
 		(stroke
@@
 	(wire
 		(pts
-			(xy 68.58 101.6) (xy 68.58 100.33)
+			(xy 142.24 38.1) (xy 139.7 38.1)
 		)
 		(stroke
@@
 	(wire
 		(pts
-			(xy 58.42 101.6) (xy 58.42 100.33)
-		)
-		(stroke
-			(width 0)
-			(type default)
-		)
-	)
-	(wire
-		(pts
 			(xy 41.91 83.82) (xy 41.91 85.09)
 		)
@@
 		)
 	)
-	(label "Q10_3"
-		(at 118.11 104.14 180)
-		(effects
-			(font
-				(size 1.27 1.27)
-			)
-			(justify right bottom)
-		)
-	)
 	(label "BIAS"
 		(at 160.02 38.1 270)
@@
 		)
 	)
-	(label "SW_C"
-		(at 68.58 101.6 180)
-		(effects
-			(font
-				(size 1.27 1.27)
-			)
-			(justify right bottom)
-		)
-	)
-	(label "Q9_3"
-		(at 76.2 92.71 180)
-		(effects
-			(font
-				(size 1.27 1.27)
-			)
-			(justify right bottom)
-		)
-	)
 	(label "VC"
 		(at 96.52 17.78 270)
@@
 		)
 	)
-	(label "Q8_3"
-		(at 50.8 91.44 0)
-		(effects
-			(font
-				(size 1.27 1.27)
-			)
-			(justify left bottom)
-		)
-	)
 	(label "BP_OUT"
 		(at 133.35 121.92 90)
@@
 		)
 	)
-	(label "Q11_3"
-		(at 128.27 104.14 0)
-		(effects
-			(font
-				(size 1.27 1.27)
-			)
-			(justify left bottom)
-		)
-	)
-	(label "SW_A"
-		(at 58.42 101.6 0)
-		(effects
-			(font
-				(size 1.27 1.27)
-			)
-			(justify left bottom)
-		)
-	)
 	(global_label "VC"
 		(shape input)
@@
 		(in_pos_files yes)
 		(dnp no)
-		(property "Reference" "Q6"
+		(property "Reference" "Q5"
 			(at 127 34.29 0)
 			(show_name no)
@@
 			(project "AMP-MA"
 				(path "/4094031b-a9da-4ac5-aaa1-42b342c92a3e/d432553b-ab0c-45ec-bbdd-5af2e9267855"
-					(reference "Q6")
+					(reference "Q5")
 					(unit 1)
 				)
@@
 		(in_pos_files yes)
 		(dnp no)
-		(property "Reference" "Q10"
+		(property "Reference" "Q11"
 			(at 116.84 89.154 90)
 			(show_name no)
@@
 			(project "AMP-MA"
 				(path "/4094031b-a9da-4ac5-aaa1-42b342c92a3e/d432553b-ab0c-45ec-bbdd-5af2e9267855"
-					(reference "Q10")
+					(reference "Q11")
 					(unit 1)
 				)
@@
 		(in_pos_files yes)
 		(dnp no)
-		(property "Reference" "Q7"
+		(property "Reference" "Q6"
 			(at 150.622 34.036 0)
 			(show_name no)
@@
 			(project "AMP-MA"
 				(path "/4094031b-a9da-4ac5-aaa1-42b342c92a3e/d432553b-ab0c-45ec-bbdd-5af2e9267855"
-					(reference "Q7")
+					(reference "Q6")
 					(unit 1)
 				)
@@
 		(in_pos_files yes)
 		(dnp no)
-		(property "Reference" "Q11"
+		(property "Reference" "Q10"
 			(at 129.54 89.408 90)
 			(show_name no)
@@
 			(project "AMP-MA"
 				(path "/4094031b-a9da-4ac5-aaa1-42b342c92a3e/d432553b-ab0c-45ec-bbdd-5af2e9267855"
-					(reference "Q11")
+					(reference "Q10")
 					(unit 1)
 				)
@@
 		(in_pos_files yes)
 		(dnp no)
-		(property "Reference" "Q9"
+		(property "Reference" "Q7"
 			(at 80.518 88.646 0)
 			(show_name no)
@@
 			(project "AMP-MA"
 				(path "/4094031b-a9da-4ac5-aaa1-42b342c92a3e/d432553b-ab0c-45ec-bbdd-5af2e9267855"
-					(reference "Q9")
+					(reference "Q7")
 					(unit 1)
 				)
@@
 		(in_pos_files yes)
 		(dnp no)
-		(property "Reference" "Q5"
+		(property "Reference" "Q4"
 			(at 127 42.164 0)
 			(show_name no)
@@
 			(project "AMP-MA"
 				(path "/4094031b-a9da-4ac5-aaa1-42b342c92a3e/d432553b-ab0c-45ec-bbdd-5af2e9267855"
-					(reference "Q5")
+					(reference "Q4")
 					(unit 1)
 				)
